File: hardware/pulse/pulse.kicad_pcb (KiCad board)
At the start: 4 copper layers, 180 x 35 mm, 170 parts, among them J1001 WAGO-2065, J1002 WAGO-2065, J101 CORTEX-DEBUG, J1101 WAGO-2065, J1102 WAGO-2065, J1201 WAGO-2065, J1202 WAGO-2065, J1301 WAGO-2065, J1302 WAGO-2065, J1401 WAGO-2065, J1402 WAGO-2065, J1501 WAGO-2065, J1502 WAGO-2065, J1601 WAGO-2065, J1602 WAGO-2065, J1701 WAGO-2065, J1702 WAGO-2065, J1801 WAGO-2065, J1802 WAGO-2065, J1901 2x05_Horizontal, J2001 2x05_Horizontal, J201 WAGO-2065, J202 WAGO-2065, J301 WAGO-2065, J302 WAGO-2065, J401 WAGO-2065, J402 WAGO-2065, J501 WAGO-2065, J502 WAGO-2065, J601 WAGO-2065, J602 WAGO-2065, J701 WAGO-2065, J702 WAGO-2065, J801 WAGO-2065, J802 WAGO-2065, J901 WAGO-2065, J902 WAGO-2065, Q1001 BSC010N04LS, Q1101 BSC010N04LS, Q1201 BSC010N04LS, Q1301 BSC010N04LS, Q1401 BSC010N04LS, Q1501 BSC010N04LS, Q1601 BSC010N04LS, Q1701 BSC010N04LS, Q201 BSC010N04LS, Q301 BSC010N04LS, Q401 BSC010N04LS, Q501 BSC010N04LS, Q601 BSC010N04LS, Q701 BSC010N04LS, Q801 BSC010N04LS, Q901 BSC010N04LS, SW101 SW_Push, SW102 SW_Push, U101 ATSAMD51J, U102 TPS78433QWDRBRQ1, U1801 BTT6010, U1901 THVD24x2, U2001 THVD24x2, Y101 32k768

Commit message: Update parts
Parts:
- C1001, C101, C102, C103, C104, C105, C106, C107, C108, C1101, C1201, C1301, C1401, C1501, C1601, C1701, C1802, C1803, C1804, C1805, C1806, C1807, C1901, C2001, C201, C301, C401, C501, C601, C701, C801, C901: footprint Capacitor_SMD:C_0603_1608Metric -> V2_Capacitor_SMD:C_0603
- C109, C110: footprint Capacitor_SMD:C_0603_1608Metric -> V2_Capacitor_SMD:C_0805
- C1801: footprint Capacitor_SMD:C_1210_3225Metric -> V2_Capacitor_SMD:C_1210
- D1001, D1101, D1201, D1301, D1401, D1501, D1601, D1701, D201, D301, D401, D501, D601, D701, D801, D901: footprint Diode_SMD:D_SOD-123F -> V2_Diode_SMD:D_SOD-123F
- D101: footprint LED_SMD:LED_0603_1608Metric -> V2_LED:LED_0603
- D1801: footprint Diode_SMD:D_SOD-523 -> V2_Diode_SMD:D_SOD-523
- FID101, FID102, FID103: value Fiducial -> Fiducial_Paste
- INFO102: value ORDER-NUMBER -> Order_Number
- J1001, J1002, J1101, J1102, J1201, J1202, J1301, J1302, J1401, J1402, J1501, J1502, J1601, J1602, J1701, J1702, J1801, J1802, J201, J202, J301, J302, J401, J402, J501, J502, J601, J602, J701, J702, J801, J802, J901, J902: value WAGO-2065 -> WAGO 2065-100
- J101: value CORTEX-DEBUG -> Cortex_Debug
- R101, R102, R1801, R1802, R1803, R1805, R1808, R1809, R1810, R1901, R2001: footprint Resistor_SMD:R_0603_1608Metric -> V2_Resistor_SMD:R_0603
- R1804: renamed from R1806; footprint Resistor_SMD:R_0603_1608Metric -> V2_Resistor_SMD:R_0603
- R1806: renamed from R1807; footprint Resistor_SMD:R_0603_1608Metric -> V2_Resistor_SMD:R_0603
- R1807: renamed from R1804; footprint Resistor_SMD:R_0603_1608Metric -> V2_Resistor_SMD:R_0603
- SW101, SW102: value SW_Push -> SKSG
- TVS101: footprint Diode_SMD:D_0603_1608Metric -> V2_Diode_SMD:D_0603
- TVS1801: value SMAJ36CA -> SMBJ36CA; footprint Diode_SMD:D_SMA -> V2_Diode_SMD:D_SMB
- U1901, U2001: value THVD24x2 -> THVD2442
- moved TVS101 0.50 mm to (69.8, 103.2)
- moved C109 0.25 mm to (69.8, 101.2)
- moved C110 0.25 mm to (69.8, 94.8)
- renumbered H102 to H101, H101 to H102
Routing:
- net /LED1: track 23.3 -> 24.6 mm

Commit message: Update library
Parts:
- J101: value Cortex_Debug -> Cortex; footprint V2_Cortex_Debug:Cortex_Debug_Pad -> V2_Connector_Debug:Cortex
- TVS1801: value SMBJ36CA -> SMBJ33CA
Connections:
- net +24V renamed +28V
Routing:
- net /SWCLK: track 11.7 -> 13.5 mm
- net GND: vias 199 -> 197
- net +3V3: vias 14 -> 13
