File: hardware/pulse/pulse.kicad_pcb (KiCad board)
At the start: 4 copper layers, 180 x 35 mm, 170 parts, among them J1001 WAGO 2065-100, J1002 WAGO 2065-100, J101 Cortex, J1101 WAGO 2065-100, J1102 WAGO 2065-100, J1201 WAGO 2065-100, J1202 WAGO 2065-100, J1301 WAGO 2065-100, J1302 WAGO 2065-100, J1401 WAGO 2065-100, J1402 WAGO 2065-100, J1501 WAGO 2065-100, J1502 WAGO 2065-100, J1601 WAGO 2065-100, J1602 WAGO 2065-100, J1701 WAGO 2065-100, J1702 WAGO 2065-100, J1801 WAGO 2065-100, J1802 WAGO 2065-100, J1901 2x05_Horizontal, J2001 2x05_Horizontal, J201 WAGO 2065-100, J202 WAGO 2065-100, J301 WAGO 2065-100, J302 WAGO 2065-100, J401 WAGO 2065-100, J402 WAGO 2065-100, J501 WAGO 2065-100, J502 WAGO 2065-100, J601 WAGO 2065-100, J602 WAGO 2065-100, J701 WAGO 2065-100, J702 WAGO 2065-100, J801 WAGO 2065-100, J802 WAGO 2065-100, J901 WAGO 2065-100, J902 WAGO 2065-100, Q1001 BSC010N04LS, Q1101 BSC010N04LS, Q1201 BSC010N04LS, Q1301 BSC010N04LS, Q1401 BSC010N04LS, Q1501 BSC010N04LS, Q1601 BSC010N04LS, Q1701 BSC010N04LS, Q201 BSC010N04LS, Q301 BSC010N04LS, Q401 BSC010N04LS, Q501 BSC010N04LS, Q601 BSC010N04LS, Q701 BSC010N04LS, Q801 BSC010N04LS, Q901 BSC010N04LS, SW101 SKSG, SW102 SKSG, U101 ATSAMD51J, U102 TPS78433QWDRBRQ1, U1801 BTT6010, U1901 THVD2442, U2001 THVD2442, Y101 32k768

Commit message: Update
Parts:
- renumbered C107 to C101, C108 to C102, C109 to C103, C101 to C104, C110 to C105, C102 to C106, C103 to C107, C104 to C108, C105 to C109, C106 to C110, C1807 to C1801, C1801 to C1802, C1802 to C1803, C1803 to C1806, C1806 to C1807, D102 to D101, D101 to D102, H103 to H102, H105 to H103, H107 to H104, H108 to H105, H102 to H106, H104 to H107, H106 to H108, ICON105 to ICON101, ICON104 to ICON102, ICON101 to ICON103, ICON102 to ICON104, ICON103 to ICON105, R102 to R101, R101 to R102, R1807 to R1801, R1806 to R1802, R1808 to R1803, R1809 to R1804, R1810 to R1805, R1804 to R1806, R1801 to R1807, R1803 to R1808, R1805 to R1809, R1802 to R1810, SW102 to SW101, SW101 to SW102, U102 to U101, U101 to U102

Commit message: Switch to 6 layer
Parts:
- C1001, C101, C102, C104, C106, C107, C108, C109, C110, C1101, C1201, C1301, C1401, C1501, C1601, C1701, C1801, C1803, C1804, C1805, C1806, C1807, C1901, C2001, C201, C301, C401, C501, C601, C701, C801, C901: footprint V2_Capacitor_SMD:C_0603 -> V2_Capacitor_SMD:C_1608
- C103, C105: footprint V2_Capacitor_SMD:C_0805 -> V2_Capacitor_SMD:C_2012
- C1802: footprint V2_Capacitor_SMD:C_1210 -> V2_Capacitor_SMD:C_3225
- D102: footprint V2_LED:LED_0603 -> V2_LED:LED_1608
- INFO101: value Layer_Numbers -> Layer_Numbers-6; footprint V2_Production:Layer_Numbers -> V2_Production:Layer_Numbers-6
- R101, R102, R1801, R1802, R1803, R1804, R1805, R1806, R1807, R1808, R1809, R1810, R1901, R2001: footprint V2_Resistor_SMD:R_0603 -> V2_Resistor_SMD:R_1608
- TVS101: footprint V2_Diode_SMD:D_0603 -> V2_Diode_SMD:D_1608
Connections:
- net /VDDCORE renamed /+VCORE
Routing:
- net +3V3: track 36.0 -> 270.3 mm
- net /Link Socket/TX-Y: track 6.68 -> 4.58 mm
- net /USB-: track 35.9 -> 37.3 mm
- added copper zone on B.Cu, net +5V
- added copper zone on In3.Cu, net GND
- added copper zone on In4.Cu, net GND
- removed copper zone on In2.Cu, net +3V3
- removed copper zone on In2.Cu, net +5V
- removed copper zone on In1.Cu, net /PWM Channel 1/PWM-Sink
- removed copper zone on In2.Cu, net /PWM Channel 1/PWM-Sink
- removed copper zone on In1.Cu, net /PWM Channel 10/PWM-Sink
- removed copper zone on In2.Cu, net /PWM Channel 10/PWM-Sink
- removed copper zone on In1.Cu, net /PWM Channel 11/PWM-Sink
- removed copper zone on In2.Cu, net /PWM Channel 11/PWM-Sink
- removed copper zone on In1.Cu, net /PWM Channel 12/PWM-Sink
- removed copper zone on In2.Cu, net /PWM Channel 12/PWM-Sink
- removed copper zone on In1.Cu, net /PWM Channel 13/PWM-Sink
- removed copper zone on In2.Cu, net /PWM Channel 13/PWM-Sink
- removed copper zone on In1.Cu, net /PWM Channel 14/PWM-Sink
- removed copper zone on In2.Cu, net /PWM Channel 14/PWM-Sink
- removed copper zone on In1.Cu, net /PWM Channel 15/PWM-Sink
- removed copper zone on In2.Cu, net /PWM Channel 15/PWM-Sink
- removed copper zone on In1.Cu, net /PWM Channel 16/PWM-Sink
- removed copper zone on In2.Cu, net /PWM Channel 16/PWM-Sink
- removed copper zone on In1.Cu, net /PWM Channel 2/PWM-Sink
- removed copper zone on In2.Cu, net /PWM Channel 2/PWM-Sink
- removed copper zone on In1.Cu, net /PWM Channel 3/PWM-Sink
- removed copper zone on In2.Cu, net /PWM Channel 3/PWM-Sink
- removed copper zone on In1.Cu, net /PWM Channel 4/PWM-Sink
- removed copper zone on In2.Cu, net /PWM Channel 4/PWM-Sink
- removed copper zone on In1.Cu, net /PWM Channel 5/PWM-Sink
- removed copper zone on In2.Cu, net /PWM Channel 5/PWM-Sink
- removed copper zone on In1.Cu, net /PWM Channel 6/PWM-Sink
- removed copper zone on In2.Cu, net /PWM Channel 6/PWM-Sink
- removed copper zone on In1.Cu, net /PWM Channel 7/PWM-Sink
- removed copper zone on In2.Cu, net /PWM Channel 7/PWM-Sink
- removed copper zone on In1.Cu, net /PWM Channel 8/PWM-Sink
- removed copper zone on In2.Cu, net /PWM Channel 8/PWM-Sink
- removed copper zone on In1.Cu, net /PWM Channel 9/PWM-Sink
- removed copper zone on In2.Cu, net /PWM Channel 9/PWM-Sink
- removed copper zone on In1.Cu, net /Power +28V/+28V-Supply
- removed copper zone on In2.Cu, net /Power +28V/+28V-Supply
- removed copper zone on B.Cu, net GND
- removed copper zone on In2.Cu, net GND
Other:
- copper layers 4 -> 6

Commit message: Update
Parts:
- moved ICON102 0.25 mm to (243.2, 83.2)
- renumbered C1301 to C1101, C1101 to C1301, C1701 to C1501, C1501 to C1701, D1301 to D1101, D1302 to D1102, D1101 to D1301, D1102 to D1302, D1701 to D1501, D1702 to D1502, D1501 to D1701, D1502 to D1702, J1301 to J1101, J1302 to J1102, J1101 to J1301, J1102 to J1302, J1701 to J1501, J1702 to J1502, J1501 to J1701, J1502 to J1702, Q1301 to Q1101, Q1101 to Q1301, Q1701 to Q1501, Q1501 to Q1701
Routing:
- net GND: vias 197 -> 215
