File: hardware/pulse/pulse.kicad_sch (KiCad schematic)
At the start: 44 parts, among them J101 CORTEX-DEBUG, SW101 SW_Push, SW102 SW_Push, U101 ATSAMD51J, U102 TPS78433QWDRBRQ1, Y101 32k768

Commit message: Update parts
Parts:
- C101: footprint Capacitor_SMD:C_0603_1608Metric -> V2_Capacitor_SMD:C_0603; symbol Device:C_Small -> V2_Device:C_0603_10u; Manufacturer (none) -> TDK; Mouser (none) -> 810-C1608X6S1A106M; Product (none) -> C1608X6S1A106M080AC
- C102, C103, C104, C105, C106: footprint Capacitor_SMD:C_0603_1608Metric -> V2_Capacitor_SMD:C_0603; symbol Device:C_Small -> V2_Device:C_0603_0u1; Manufacturer (none) -> TDK; Mouser (none) -> 810-CGA3E2X7R1H104MA; Product (none) -> CGA3E2X7R1H104M080AA
- C107, C108: footprint Capacitor_SMD:C_0603_1608Metric -> V2_Capacitor_SMD:C_0603; symbol Device:C_Small -> V2_Device:C_0603_18p; Manufacturer (none) -> YAGEO; Mouser (none) -> 603-CC603JRNPO9BN180; Product (none) -> CC0603JRNPO9BN180
- C109, C110: footprint Capacitor_SMD:C_0603_1608Metric -> V2_Capacitor_SMD:C_0805; symbol Device:C_Small -> V2_Device:C_0805_10u; Manufacturer (none) -> TDK; Mouser (none) -> 810-C2012X5R1E106K; Product (none) -> C2012X5R1E106K125AB; Rating (none) -> 25V
- D101: footprint LED_SMD:LED_0603_1608Metric -> V2_LED:LED_0603; symbol Device:LED_Small -> V2_Device:LED_0603_Orange; Manufacturer (none) -> ROHM Semiconductor; Mouser (none) -> 755-SML-D12M8WT86C; Product (none) -> SML-D12M8WT86C
- D102, D103: LCSC (none) -> C965555; Manufacturer (none) -> Worldsemi; Product (none) -> WS2812B-2020
- ESD101: Manufacturer (none) -> Semtech; Mouser (none) -> 947-RCLAMP0582N.TCT; Product (none) -> RCLAMP0582N.TCT
- FID101, FID102, FID103: value Fiducial -> Fiducial_Paste
- INFO102: value ORDER-NUMBER -> Order_Number
- J101: value CORTEX-DEBUG -> Cortex_Debug
- R101: footprint Resistor_SMD:R_0603_1608Metric -> V2_Resistor_SMD:R_0603; symbol Device:R_Small -> V2_Device:R_0603_330R; Manufacturer (none) -> Vishay; Mouser (none) -> 71-CRCW0603330RFKEAC; Product (none) -> CRCW0603330RFKEAC; Rating (none) -> 100mW
- R102: footprint Resistor_SMD:R_0603_1608Metric -> V2_Resistor_SMD:R_0603; symbol Device:R_Small -> V2_Device:R_0603_100k; Manufacturer (none) -> Vishay; Mouser (none) -> 71-CRCW0603100KFKEAC; Product (none) -> CRCW0603100KFKEAC; Rating (none) -> 100mW
- SW101, SW102: value SW_Push -> SKSG; symbol Switch:SW_Push -> V2_Switch:SKSG; Manufacturer (none) -> Alps Alpine; Mouser (none) -> 688-SKSGACE010; Product (none) -> SKSGACE010
- TVS101: footprint Diode_SMD:D_0603_1608Metric -> V2_Diode_SMD:D_0603; Manufacturer (none) -> Bourns; Mouser (none) -> 652-CG0603MLC-05LE; Product (none) -> CG0603MLC-05LE; Rating (none) -> 5V
- U101: Manufacturer (none) -> Microchip Technology; Mouser (none) -> 556-ATSAMD51J19AMU; Product (none) -> ATSAMD51J19A-MU
- U102: Manufacturer (none) -> Texas Instruments; Mouser (none) -> 595-TPS78433QWDRBRQ1; Product (none) -> TPS78433QWDRBRQ1
- Y101: symbol Device:Crystal_Small -> V2_Device:Crystal_3.2x1.5_32k768; Manufacturer (none) -> ABRACON; Mouser (none) -> 815-ABS0716632.768KT; Product (none) -> ABS07-166-32.768KHZ-T
- renumbered H102 to H101, H101 to H102
Other:
- moved on the sheet: FID101, FID102, FID103, H102, H104, H106

Commit message: Refresh
Parts:
- D101: Mouser 755-SML-D12M8WT86C -> 755-SML-D12D1WT86; Product SML-D12M8WT86C -> SML-D12D1WT86

Commit message: Update library
Parts:
- C101: Rating (none) -> 10V
- C102, C103, C104, C105, C106: Rating (none) -> 50V
- J101: value Cortex_Debug -> Cortex; footprint V2_Cortex_Debug:Cortex_Debug_Pad -> V2_Connector_Debug:Cortex; symbol V2_Cortex_Debug:Cortex_Debug -> V2_Connector_Debug:Cortex
Changed lines of the file:
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@@
 			)
 		)
-		(property "Description" "Power symbol creates a global label with name \"+5V\""
+		(property "Description" ""
 			(at 179.07 125.73 0)
 			(effects
@@
 			)
 		)
-		(property "Description" "Power symbol creates a global label with name \"+5V\""
+		(property "Description" ""
 			(at 195.58 121.92 0)
 			(effects
@@
 			)
 		)
+		(property "Rating" "50V"
+			(at 109.22 46.99 0)
+			(effects
+				(font
+					(size 1.27 1.27)
+				)
+				(hide yes)
+			)
+		)
 		(pin "1"
 		)
@@
 			)
 		)
-		(property "Description" "Power symbol creates a global label with name \"GND\" , ground"
+		(property "Description" ""
 			(at 133.35 186.69 0)
 			(effects
@@
 			)
 		)
-		(property "Description" "Power symbol creates a global label with name \"+3V3\""
+		(property "Description" ""
 			(at 58.42 166.37 0)
 			(effects
@@
 			)
 		)
-		(property "Description" "Power symbol creates a global label with name \"GND\" , ground"
+		(property "Description" ""
 			(at 58.42 171.45 0)
 			(effects
@@
 			)
 		)
-		(property "Description" "Power symbol creates a global label with name \"GND\" , ground"
+		(property "Description" ""
 			(at 67.31 127 0)
 			(effects
@@
 			)
 		)
-		(property "Description" "Power symbol creates a global label with name \"GND\" , ground"
+		(property "Description" ""
 			(at 26.67 49.53 0)
 			(effects
@@
 			)
 		)
-		(property "Description" "Power symbol creates a global label with name \"GND\" , ground"
+		(property "Description" ""
 			(at 57.15 26.67 0)
 			(effects
@@
 			)
 		)
-		(property "Description" "Power symbol creates a global label with name \"+3V3\""
+		(property "Description" ""
 			(at 72.39 21.59 0)
 			(effects
@@
 			)
 		)
-		(property "Description" "Power symbol creates a global label with name \"+5V\""
+		(property "Description" ""
 			(at 133.35 173.99 0)
 			(effects
@@
 			)
 		)
-		(property "Description" "Power symbol creates a global label with name \"+3V3\""
+		(property "Description" ""
 			(at 48.26 121.92 0)
 			(effects
@@
 			)
 		)
+		(property "Rating" "50V"
+			(at 119.38 46.99 0)
+			(effects
+				(font
+					(size 1.27 1.27)
+				)
+				(hide yes)
+			)
+		)
 		(pin "1"
 		)
@@
 	)
 	(symbol
-		(lib_id "V2_Cortex_Debug:Cortex_Debug")
+		(lib_id "V2_Connector_Debug:Cortex")
 		(at 124.46 107.95 0)
 		(unit 1)
@@
 			)
 		)
-		(property "Value" "Cortex_Debug"
-			(at 125.73 97.79 0)
+		(property "Value" "Cortex"
+			(at 115.57 99.06 0)
 			(effects
 				(font
 					(size 1.27 1.27)
 				)
+				(justify left bottom)
 			)
 		)
-		(property "Footprint" "V2_Cortex_Debug:Cortex_Debug_Pad"
+		(property "Footprint" "V2_Connector_Debug:Cortex"
 			(at 124.46 121.92 0)
 			(effects
@@
 			)
 		)
-		(property "Sim.Enable" "0"
-			(at 124.46 107.95 0)
-			(effects
-				(font
-					(size 1.27 1.27)
-				)
-				(hide yes)
-			)
-		)
 		(pin "1"
 		)
@@
 			)
 		)
-		(property "Description" "Power symbol creates a global label with name \"GND\" , ground"
+		(property "Description" ""
 			(at 21.59 49.53 0)
 			(effects
@@
 			)
 		)
-		(property "Description" "Power symbol creates a global label with name \"GND\" , ground"
+		(property "Description" ""
 			(at 113.03 113.03 0)
 			(effects
@@
 			)
 		)
-		(property "Description" "Power symbol creates a global label with name \"GND\" , ground"
+		(property "Description" ""
 			(at 179.07 128.27 0)
 			(effects
@@
 			)
 		)
-		(property "Description" "Power symbol creates a global label with name \"+5V\""
+		(property "Description" ""
 			(at 33.02 166.37 0)
 			(effects
@@
 			)
 		)
-		(property "Description" "Power symbol creates a global label with name \"+3V3\""
+		(property "Description" ""
 			(at 53.34 48.26 0)
 			(effects
@@
 			)
 		)
-		(property "Description" "Power symbol creates a global label with name \"GND\" , ground"
+		(property "Description" ""
 			(at 78.74 26.67 0)
 			(effects
@@
 			)
 		)
-		(property "Description" "Power symbol creates a global label with name \"GND\" , ground"
+		(property "Description" ""
 			(at 266.7 118.11 0)
 			(effects
@@
 			)
 		)
-		(property "Description" "Power symbol creates a global label with name \"GND\" , ground"
+		(property "Description" ""
 			(at 113.03 157.48 0)
 			(effects
@@
 			)
 		)
-		(property "Description" "Power symbol creates a global label with name \"+3V3\""
+		(property "Description" ""
 			(at 113.03 102.87 0)
 			(effects
@@
 			)
 		)
+		(property "Rating" "10V"
+			(at 57.15 49.53 0)
+			(effects
+				(font
+					(size 1.27 1.27)
+				)
+				(hide yes)
+			)
+		)
 		(pin "1"
 		)
@@
 			)
 		)
-		(property "Description" "Power symbol creates a global label with name \"GND\" , ground"
+		(property "Description" ""
 			(at 33.02 171.45 0)
 			(effects
@@
 			)
 		)
-		(property "Description" "Power symbol creates a global label with name \"GND\" , ground"
+		(property "Description" ""
 			(at 45.72 176.53 0)
 			(effects
@@
 			)
 		)
-		(property "Description" "Power symbol creates a global label with name \"GND\" , ground"
+		(property "Description" ""
 			(at 137.16 86.36 0)
 			(effects
@@
 			)
 		)
+		(property "Rating" "50V"
+			(at 99.06 46.99 0)
+			(effects
+				(font
+					(size 1.27 1.27)
+				)
+				(hide yes)
+			)
+		)
 		(pin "1"
 		)
@@
 			)
 		)
+		(property "Rating" "50V"
+			(at 78.74 46.99 0)
+			(effects
+				(font
+					(size 1.27 1.27)
+				)
+				(hide yes)
+			)
+		)
 		(pin "1"
 		)
@@
 			)
 		)
-		(property "Description" "Power symbol creates a global label with name \"GND\" , ground"
+		(property "Description" ""
 			(at 86.36 48.26 0)
 			(effects
@@
 			)
 		)
-		(property "Description" "Power symbol creates a global label with name \"GND\" , ground"
+		(property "Description" ""
 			(at 195.58 129.54 0)
 			(effects
@@
 			)
 		)
-		(property "Description" "Power symbol creates a global label with name \"GND\" , ground"
+		(property "Description" ""
 			(at 128.27 67.31 0)
 			(effects
@@
 			)
 		)
-		(property "Description" "Power symbol creates a global label with name \"GND\" , ground"
+		(property "Description" ""
 			(at 227.33 118.11 0)
 			(effects
@@
 			(effects
 				(font
+					(size 1.27 1.27)
+				)
+				(hide yes)
+			)
+		)
+		(property "Rating" "50V"
+			(at 88.9 46.99 0)
+			(effects
+				(font
