File: hardware/pulse/pulse.kicad_sch (KiCad schematic)
At the start: 44 parts, among them J101 Cortex, SW101 SKSG, SW102 SKSG, U101 TPS78433QWDRBRQ1, U102 ATSAMD51J, Y101 32k768

Commit message: Rename
Connections:
- net +5V: now also U101.6 (EN)
Other:
- sheet Link Plug: file LinkPlug.kicad_sch -> Link-Plug.kicad_sch
- sheet Link Socket: file LinkSocket.kicad_sch -> Link-Socket.kicad_sch
- sheet PWM Channel 1: file PWMChannel.kicad_sch -> PWM-Channel.kicad_sch
- sheet PWM Channel 10: file PWMChannel.kicad_sch -> PWM-Channel.kicad_sch
- sheet PWM Channel 11: file PWMChannel.kicad_sch -> PWM-Channel.kicad_sch
- sheet PWM Channel 12: file PWMChannel.kicad_sch -> PWM-Channel.kicad_sch
- sheet PWM Channel 13: file PWMChannel.kicad_sch -> PWM-Channel.kicad_sch
- sheet PWM Channel 14: file PWMChannel.kicad_sch -> PWM-Channel.kicad_sch
- sheet PWM Channel 15: file PWMChannel.kicad_sch -> PWM-Channel.kicad_sch
- sheet PWM Channel 16: file PWMChannel.kicad_sch -> PWM-Channel.kicad_sch
- sheet PWM Channel 2: file PWMChannel.kicad_sch -> PWM-Channel.kicad_sch
- sheet PWM Channel 3: file PWMChannel.kicad_sch -> PWM-Channel.kicad_sch
- sheet PWM Channel 4: file PWMChannel.kicad_sch -> PWM-Channel.kicad_sch
- sheet PWM Channel 5: file PWMChannel.kicad_sch -> PWM-Channel.kicad_sch
- sheet PWM Channel 6: file PWMChannel.kicad_sch -> PWM-Channel.kicad_sch
- sheet PWM Channel 7: file PWMChannel.kicad_sch -> PWM-Channel.kicad_sch
- sheet PWM Channel 8: file PWMChannel.kicad_sch -> PWM-Channel.kicad_sch
- sheet PWM Channel 9: file PWMChannel.kicad_sch -> PWM-Channel.kicad_sch
- sheet Power +28V: file PowerSwitch.kicad_sch -> Power-Switch.kicad_sch
