File: hardware/pulse/PowerSwitch.kicad_sch (KiCad schematic)
At the start: 22 parts, among them J1801 WAGO-2065, J1802 WAGO-2065, U1801 BTT6010

Commit message: Update parts
Parts:
- C1801: footprint Capacitor_SMD:C_1210_3225Metric -> V2_Capacitor_SMD:C_1210; symbol Device:C_Small -> V2_Device:C_1210_10u; Manufacturer (none) -> TDK; Mouser (none) -> 810-CNA6P1X7R1H106K2; Product (none) -> CNA6P1X7R1H106K250AE; Rating (none) -> 50V; Voltage (none) -> 50V
- C1802, C1803, C1804, C1805, C1806, C1807: footprint Capacitor_SMD:C_0603_1608Metric -> V2_Capacitor_SMD:C_0603; symbol Device:C_Small -> V2_Device:C_0603_0u1; Manufacturer (none) -> TDK; Mouser (none) -> 810-CGA3E2X7R1H104MA; Product (none) -> CGA3E2X7R1H104M080AA
- D1801: footprint Diode_SMD:D_SOD-523 -> V2_Diode_SMD:D_SOD-523; Manufacturer (none) -> ROHM Semiconductor; Mouser (none) -> 755-RB501SM-30FHT2R; Product (none) -> RB501SM-30FHT2R
- J1801, J1802: value WAGO-2065 -> WAGO 2065-100; Manufacturer (none) -> WAGO; Product (none) -> 2065-100/998-403
- R1801: footprint Resistor_SMD:R_0603_1608Metric -> V2_Resistor_SMD:R_0603; symbol Device:R_Small -> V2_Device:R_0603_100k; Manufacturer (none) -> Vishay; Mouser (none) -> 71-CRCW0603100KFKEAC; Product (none) -> CRCW0603100KFKEAC; Rating (none) -> 100mW
- R1802, R1803, R1808: footprint Resistor_SMD:R_0603_1608Metric -> V2_Resistor_SMD:R_0603; symbol Device:R_Small -> V2_Device:R_0603_10k; Manufacturer (none) -> Vishay; Mouser (none) -> 71-CRCW060310K0FKEAC; Product (none) -> CRCW060310K0FKEAC; Rating (none) -> 100mW
- R1804: renamed from R1806; footprint Resistor_SMD:R_0603_1608Metric -> V2_Resistor_SMD:R_0603; symbol Device:R_Small -> V2_Device:R_0603_100k; Manufacturer (none) -> Vishay; Mouser (none) -> 71-CRCW0603100KFKEAC; Product (none) -> CRCW0603100KFKEAC; Rating (none) -> 100mW
- R1805: footprint Resistor_SMD:R_0603_1608Metric -> V2_Resistor_SMD:R_0603; symbol Device:R_Small -> V2_Device:R_0603_100R; Manufacturer (none) -> Vishay; Mouser (none) -> 71-CRCW0603100RFKEAH; Product (none) -> CRCW0603100RFKEAHP; Rating (none) -> 330mW
- R1806: renamed from R1807; footprint Resistor_SMD:R_0603_1608Metric -> V2_Resistor_SMD:R_0603; symbol Device:R_Small -> V2_Device:R_0603_10k; Manufacturer (none) -> Vishay; Mouser (none) -> 71-CRCW060310K0FKEAC; Product (none) -> CRCW060310K0FKEAC; Rating (none) -> 100mW
- R1807: renamed from R1804; footprint Resistor_SMD:R_0603_1608Metric -> V2_Resistor_SMD:R_0603; symbol Device:R_Small -> V2_Device:R_0603_100k; Manufacturer (none) -> Vishay; Mouser (none) -> 71-CRCW0603100KFKEAC; Product (none) -> CRCW0603100KFKEAC; Rating (none) -> 100mW
- R1809, R1810: footprint Resistor_SMD:R_0603_1608Metric -> V2_Resistor_SMD:R_0603; symbol Device:R_Small -> V2_Device:R_0603_2k7; Manufacturer (none) -> Vishay; Mouser (none) -> 71-CRCW06032K70FKEAC; Product (none) -> CRCW06032K70FKEAC; Rating (none) -> 100mW
- TVS1801: value SMAJ36CA -> SMBJ36CA; footprint Diode_SMD:D_SMA -> V2_Diode_SMD:D_SMB; symbol V2_Diode:SMAJ36CA -> V2_Diode:SMBJ36CA; Manufacturer (none) -> Bourns; Mouser (none) -> 652-SMBJ36CA-Q; Product (none) -> SMBJ36CA-Q; Rating (none) -> 36V
- U1801: Manufacturer (none) -> Infineon; Mouser (none) -> 726-BTT60101ERBXUMA1; Product (none) -> BTT60101ERBXUMA1
Other:
- moved on the sheet: C1804, C1805, R1801, R1804, R1805, R1806, R1807, R1808, R1809, R1810, U1801

Commit message: Refresh
Parts:
- C1801: Rating 50V -> (none)

Commit message: Update library
Parts:
- C1801: Rating (none) -> 50V; Voltage 50V -> (none)
- C1802, C1803, C1804, C1805, C1806, C1807: Rating (none) -> 50V
- TVS1801: value SMBJ36CA -> SMBJ33CA; symbol V2_Diode:SMBJ36CA -> V2_Diode:SMBJ33CA; Mouser 652-SMBJ36CA-Q -> 652-SMBJ33CA-Q; Product SMBJ36CA-Q -> SMBJ33CA-Q; Rating 36V -> 33V
Connections:
- net +24V renamed +28V
Changed lines of the file:
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@@
 			)
 		)
-		(property "Description" "Power symbol creates a global label with name \"GND\" , ground"
+		(property "Description" ""
 			(at 102.87 83.82 0)
 			(effects
@@
 			)
 		)
-		(property "Description" "Power symbol creates a global label with name \"GND\" , ground"
+		(property "Description" ""
 			(at 218.44 81.28 0)
 			(effects
@@
 			)
 		)
-		(property "Voltage" "50V"
-			(at 120.65 99.06 0)
+		(property "Product" "CNA6P1X7R1H106K250AE"
+			(at 120.65 96.52 0)
 			(effects
 				(font
@@
 			)
 		)
-		(property "Product" "CNA6P1X7R1H106K250AE"
-			(at 120.65 96.52 0)
+		(property "Manufacturer" "TDK"
+			(at 120.65 93.98 0)
 			(effects
 				(font
@@
 			)
 		)
-		(property "Manufacturer" "TDK"
-			(at 120.65 93.98 0)
+		(property "Rating" "50V"
+			(at 120.65 99.06 0)
 			(effects
 				(font
@@
 			)
 		)
-		(property "Description" "Power symbol creates a global label with name \"GND\" , ground"
+		(property "Description" ""
 			(at 132.08 81.28 0)
 			(effects
@@
 			)
 		)
-		(property "Description" "Power symbol creates a global label with name \"GND\" , ground"
+		(property "Description" ""
 			(at 107.95 140.97 0)
 			(effects
@@
 			)
 		)
-		(property "Description" "Power symbol creates a global label with name \"GND\" , ground"
+		(property "Description" ""
 			(at 154.94 125.73 0)
 			(effects
@@
 	)
 	(symbol
-		(lib_id "V2_Diode:SMBJ36CA")
+		(lib_id "V2_Diode:SMBJ33CA")
 		(at 102.87 80.01 90)
 		(unit 1)
@@
 			)
 		)
-		(property "Value" "SMBJ36CA"
+		(property "Value" "SMBJ33CA"
 			(at 111.125 81.2799 90)
 			(effects
@@
 			)
 		)
-		(property "Description" ""
+		(property "Description" "Transient Voltage Suppressor Diode, Bidirectional, 36.7-40.6V"
 			(at 102.87 80.01 0)
 			(effects
@@
 			)
 		)
-		(property "Mouser" "652-SMBJ36CA-Q"
+		(property "Mouser" "652-SMBJ33CA-Q"
 			(at 110.236 80.01 0)
 			(effects
@@
 			)
 		)
-		(property "Product" "SMBJ36CA-Q"
+		(property "Product" "SMBJ33CA-Q"
 			(at 113.03 80.01 0)
 			(effects
@@
 			)
 		)
-		(property "Rating" "36V"
+		(property "Rating" "33V"
 			(at 115.57 80.01 0)
 			(effects
@@
 			)
 		)
-		(property "Description" "Power symbol creates a global label with name \"GND\" , ground"
+		(property "Description" ""
 			(at 85.09 130.81 0)
 			(effects
@@
 			)
 		)
-		(property "Description" "Power symbol creates a global label with name \"GND\" , ground"
+		(property "Description" ""
 			(at 217.17 130.81 0)
 			(effects
@@
 			)
 		)
-		(property "Description" "Power symbol creates a global label with name \"+3V3\""
+		(property "Description" ""
 			(at 199.39 120.65 0)
 			(effects
@@
 			)
 		)
-		(property "Description" "Power symbol creates a global label with name \"GND\" , ground"
+		(property "Description" ""
 			(at 137.16 135.89 0)
 			(effects
@@
 			)
 		)
+		(property "Rating" "50V"
+			(at 154.94 146.05 0)
+			(effects
+				(font
+					(size 1.27 1.27)
+				)
+				(hide yes)
+			)
+		)
 		(pin "1"
 		)
@@
 			)
 		)
-		(property "Description" "Power symbol creates a global label with name \"GND\" , ground"
+		(property "Description" ""
 			(at 120.65 81.28 0)
 			(effects
@@
 	)
 	(symbol
-		(lib_id "V2_power:+24V")
+		(lib_id "V2_power:+28V")
 		(at 167.64 120.65 0)
 		(unit 1)
@@
 			)
 		)
-		(property "Value" "+24V"
+		(property "Value" "+28V"
 			(at 167.64 115.57 0)
 			(effects
@@
 			)
 		)
-		(property "Description" "Power symbol creates a global label with name \"+24V\""
+		(property "Description" ""
 			(at 167.64 120.65 0)
 			(effects
@@
 	)
 	(symbol
-		(lib_id "V2_power:+24V")
+		(lib_id "V2_power:+28V")
 		(at 199.39 130.81 180)
 		(unit 1)
@@
 			)
 		)
-		(property "Value" "+24V"
+		(property "Value" "+28V"
 			(at 199.39 135.89 0)
 			(effects
@@
 			)
 		)
-		(property "Description" "Power symbol creates a global label with name \"+24V\""
+		(property "Description" ""
 			(at 199.39 130.81 0)
 			(effects
@@
 			)
 		)
-		(property "Description" "Power symbol creates a global label with name \"GND\" , ground"
+		(property "Description" ""
 			(at 116.84 140.97 0)
 			(effects
@@
 			)
 		)
+		(property "Rating" "50V"
+			(at 132.08 101.6 0)
+			(effects
+				(font
+					(size 1.27 1.27)
+				)
+				(hide yes)
+			)
+		)
 		(pin "1"
 		)
@@
 			)
 		)
-		(property "Description" "Power symbol creates a global label with name \"GND\" , ground"
+		(property "Description" ""
 			(at 193.04 81.28 0)
 			(effects
@@
 			)
 		)
-		(property "Description" "Power symbol creates a global label with name \"GND\" , ground"
+		(property "Description" ""
 			(at 167.64 125.73 0)
 			(effects
@@
 			)
 		)
-		(property "Description" "Power symbol creates a global label with name \"GND\" , ground"
+		(property "Description" ""
 			(at 142.24 125.73 0)
 			(effects
@@
 			)
 		)
+		(property "Rating" "50V"
+			(at 85.09 161.29 0)
+			(effects
+				(font
+					(size 1.27 1.27)
+				)
+				(hide yes)
+			)
+		)
 		(pin "1"
 		)
@@
 			)
 		)
-		(property "Description" "Power symbol creates a global label with name \"GND\" , ground"
+		(property "Description" ""
 			(at 85.09 140.97 0)
 			(effects
@@
 			)
 		)
+		(property "Rating" "50V"
+			(at 217.17 151.13 0)
+			(effects
+				(font
+					(size 1.27 1.27)
+				)
+				(hide yes)
+			)
+		)
 		(pin "1"
 		)
@@
 			)
 		)
+		(property "Rating" "50V"
+			(at 167.64 146.05 0)
+			(effects
+				(font
+					(size 1.27 1.27)
+				)
+				(hide yes)
+			)
+		)
 		(pin "1"
 		)
@@
 			)
 		)
+		(property "Rating" "50V"
+			(at 218.44 101.6 0)
+			(effects
+				(font
+					(size 1.27 1.27)
+				)
+				(hide yes)
+			)
+		)
 		(pin "1"
 		)
@@
 			)
 		)
-		(property "Description" "Power symbol creates a global label with name \"+3V3\""
+		(property "Description" ""
 			(at 116.84 130.81 0)
 			(effects

Commit message: Update Library
Parts:
- C1801: symbol V2_Device:C_1210_10u -> V2_Capacitor:1210_10u
- C1802, C1803, C1804, C1805, C1806, C1807: symbol V2_Device:C_0603_0u1 -> V2_Capacitor:0603_0u1
- R1801, R1804, R1807: symbol V2_Device:R_0603_100k -> V2_Resistor:0603_100k
- R1802, R1803, R1806, R1808: symbol V2_Device:R_0603_10k -> V2_Resistor:0603_10k
- R1805: symbol V2_Device:R_0603_100R -> V2_Resistor:0603_100R
- R1809, R1810: symbol V2_Device:R_0603_2k7 -> V2_Resistor:0603_2k7
Changed lines of the file:
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@@
 	)
 	(symbol
-		(lib_id "V2_Device:C_1210_10u")
+		(lib_id "V2_Capacitor:1210_10u")
 		(at 120.65 78.74 0)
 		(unit 1)
@@
 	)
 	(symbol
-		(lib_id "V2_Device:R_0603_10k")
+		(lib_id "V2_Resistor:0603_10k")
 		(at 92.71 125.73 270)
 		(unit 1)
@@
 	)
 	(symbol
-		(lib_id "V2_Device:R_0603_10k")
+		(lib_id "V2_Resistor:0603_10k")
 		(at 92.71 135.89 90)
 		(unit 1)
@@
 	)
 	(symbol
-		(lib_id "V2_Device:R_0603_10k")
+		(lib_id "V2_Resistor:0603_10k")
 		(at 208.28 76.2 90)
 		(unit 1)
@@
 	)
 	(symbol
-		(lib_id "V2_Device:R_0603_2k7")
+		(lib_id "V2_Resistor:0603_2k7")
 		(at 107.95 138.43 0)
 		(unit 1)
@@
 	)
 	(symbol
-		(lib_id "V2_Device:R_0603_10k")
+		(lib_id "V2_Resistor:0603_10k")
 		(at 193.04 78.74 0)
 		(unit 1)
@@
 	)
 	(symbol
-		(lib_id "V2_Device:R_0603_100k")
+		(lib_id "V2_Resistor:0603_100k")
 		(at 193.04 73.66 0)
 		(unit 1)
@@
 	)
 	(symbol
-		(lib_id "V2_Device:C_0603_0u1")
+		(lib_id "V2_Capacitor:0603_0u1")
 		(at 154.94 123.19 0)
 		(unit 1)
@@
 	)
 	(symbol
-		(lib_id "V2_Device:R_0603_100k")
+		(lib_id "V2_Resistor:0603_100k")
 		(at 85.09 128.27 180)
 		(unit 1)
@@
 	)
 	(symbol
-		(lib_id "V2_Device:R_0603_100k")
+		(lib_id "V2_Resistor:0603_100k")
 		(at 142.24 123.19 0)
 		(unit 1)
@@
 	)
 	(symbol
-		(lib_id "V2_Device:R_0603_100R")
+		(lib_id "V2_Resistor:0603_100R")
 		(at 199.39 123.19 0)
 		(unit 1)
@@
 	)
 	(symbol
-		(lib_id "V2_Device:C_0603_0u1")
+		(lib_id "V2_Capacitor:0603_0u1")
 		(at 132.08 78.74 0)
 		(unit 1)
@@
 	)
 	(symbol
-		(lib_id "V2_Device:R_0603_2k7")
+		(lib_id "V2_Resistor:0603_2k7")
 		(at 116.84 138.43 0)
 		(unit 1)
@@
 	)
 	(symbol
-		(lib_id "V2_Device:C_0603_0u1")
+		(lib_id "V2_Capacitor:0603_0u1")
 		(at 85.09 138.43 0)
 		(unit 1)
@@
 	)
 	(symbol
-		(lib_id "V2_Device:C_0603_0u1")
+		(lib_id "V2_Capacitor:0603_0u1")
 		(at 217.17 128.27 0)
 		(unit 1)
@@
 	)
 	(symbol
-		(lib_id "V2_Device:C_0603_0u1")
+		(lib_id "V2_Capacitor:0603_0u1")
 		(at 167.64 123.19 0)
 		(unit 1)
@@
 	)
 	(symbol
-		(lib_id "V2_Device:C_0603_0u1")
+		(lib_id "V2_Capacitor:0603_0u1")
 		(at 218.44 78.74 0)
 		(unit 1)
