File: hardware/pulse/LinkPlug.kicad_sch (KiCad schematic)
At the start: 4 parts, among them J1901 2x05_Horizontal, U1901 THVD24x2

Commit message: Update
Other:
- note added: "+5V from Plug"
- note added: "RS-422 3MHz"
- note removed: "Power input from plug."
- moved on the sheet: R1901
Changed lines of the file:
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@@
 		(company "Plug")
 	)
-	(text "Power input from plug."
+	(text "+5V from Plug"
 		(exclude_from_sim no)
-		(at 137.16 172.72 0)
+		(at 140.97 172.974 0)
 		(effects
 			(font
@@
 			)
 			(justify left bottom)
+		)
+	)
+	(text "RS-422 3MHz"
+		(exclude_from_sim no)
+		(at 168.91 88.9 0)
+		(effects
+			(font
+				(size 1.27 1.27)
+			)
 		)
 	)
@@
 		(color 0 0 0 0)
 	)
-	(wire
-		(pts
-			(xy 148.59 105.41) (xy 139.7 105.41)
-		)
-		(stroke
-			(width 0)
-			(type default)
-		)
+	(junction
+		(at 160.02 62.23)
+		(diameter 0)
+		(color 0 0 0 0)
+	)
+	(junction
+		(at 160.02 57.15)
+		(diameter 0)
+		(color 0 0 0 0)
 	)
 	(wire
@@
 	(wire
 		(pts
-			(xy 158.75 67.31) (xy 170.18 67.31)
-		)
-		(stroke
-			(width 0)
-			(type default)
-		)
-	)
-	(wire
-		(pts
-			(xy 158.75 72.39) (xy 170.18 72.39)
+			(xy 158.75 67.31) (xy 175.26 67.31)
+		)
+		(stroke
+			(width 0)
+			(type default)
+		)
+	)
+	(wire
+		(pts
+			(xy 158.75 72.39) (xy 175.26 72.39)
 		)
 		(stroke
@@
 	(wire
 		(pts
-			(xy 158.75 62.23) (xy 170.18 62.23)
+			(xy 158.75 62.23) (xy 160.02 62.23)
 		)
 		(stroke
@@
 	(wire
 		(pts
-			(xy 148.59 110.49) (xy 139.7 110.49)
-		)
-		(stroke
-			(width 0)
-			(type default)
-		)
-	)
-	(wire
-		(pts
 			(xy 142.24 138.43) (xy 128.27 138.43)
 		)
@@
 	(wire
 		(pts
-			(xy 158.75 57.15) (xy 170.18 57.15)
+			(xy 158.75 57.15) (xy 160.02 57.15)
 		)
 		(stroke
@@
 	(wire
 		(pts
+			(xy 160.02 62.23) (xy 175.26 62.23)
+		)
+		(stroke
+			(width 0)
+			(type default)
+		)
+	)
+	(wire
+		(pts
+			(xy 160.02 57.15) (xy 175.26 57.15)
+		)
+		(stroke
+			(width 0)
+			(type default)
+		)
+	)
+	(wire
+		(pts
 			(xy 154.94 143.51) (xy 172.72 143.51)
 		)
@@
 	)
 	(label "RX-B"
-		(at 170.18 62.23 180)
+		(at 175.26 62.23 180)
 		(effects
 			(font
@@
 	)
 	(label "RX-A"
-		(at 139.7 105.41 0)
-		(effects
-			(font
-				(size 1.27 1.27)
-			)
-			(justify left bottom)
-		)
-	)
-	(label "RX-A"
-		(at 170.18 57.15 180)
+		(at 175.26 57.15 180)
 		(effects
 			(font
@@
 		)
 	)
-	(label "RX-B"
-		(at 139.7 110.49 0)
-		(effects
-			(font
-				(size 1.27 1.27)
-			)
-			(justify left bottom)
-		)
-	)
 	(label "TX-Z"
-		(at 170.18 67.31 180)
+		(at 175.26 67.31 180)
 		(effects
 			(font
@@
 	)
 	(label "TX-Y"
-		(at 170.18 72.39 180)
+		(at 175.26 72.39 180)
 		(effects
 			(font
@@
 	(symbol
 		(lib_id "Device:R_Small")
-		(at 148.59 107.95 0)
+		(at 160.02 59.69 0)
 		(unit 1)
 		(exclude_from_sim no)
@@
 		(dnp no)
 		(property "Reference" "R1901"
-			(at 153.67 106.68 0)
+			(at 165.1 58.42 0)
 			(effects
 				(font
@@
 		)
 		(property "Value" "100R"
-			(at 153.67 109.22 0)
+			(at 165.1 60.96 0)
 			(effects
 				(font
@@
 		)
 		(property "Footprint" "Resistor_SMD:R_0603_1608Metric"
-			(at 148.59 107.95 0)
+			(at 160.02 59.69 0)
 			(effects
 				(font
@@
 		)
 		(property "Datasheet" "~"
-			(at 148.59 107.95 0)
+			(at 160.02 59.69 0)
 			(effects
 				(font
@@
 		)
 		(property "Description" "Resistor, small symbol"
-			(at 148.59 107.95 0)
+			(at 160.02 59.69 0)
 			(effects
 				(font
@@
 		(at 148.59 143.51 0)
 		(unit 1)
-		(exclude_from_sim no)
+		(exclude_from_sim yes)
 		(in_bom yes)
 		(on_board yes)
@@
 			(at 148.59 143.51 0)
 			(effects
-				(font
-					(size 1.27 1.27)
-				)
-				(hide yes)
-			)
-		)
-		(property "Sim.Enable" "0"
-			(at 148.59 143.51 0)
-			(effects

Commit message: Update parts
Parts:
- C1901: footprint Capacitor_SMD:C_0603_1608Metric -> V2_Capacitor_SMD:C_0603; symbol Device:C_Small -> V2_Device:C_0603_0u1; Manufacturer (none) -> TDK; Mouser (none) -> 810-CGA3E2X7R1H104MA; Product (none) -> CGA3E2X7R1H104M080AA
- J1901: Manufacturer (none) -> Amphenol FCI; Mouser (none) -> 649-200211120001T4LF; Product (none) -> 20021112-00010T4LF
- R1901: footprint Resistor_SMD:R_0603_1608Metric -> V2_Resistor_SMD:R_0603; symbol Device:R_Small -> V2_Device:R_0603_100R; Manufacturer (none) -> Vishay; Mouser (none) -> 71-CRCW0603100RFKEAH; Product (none) -> CRCW0603100RFKEAHP; Rating (none) -> 330mW
- U1901: value THVD24x2 -> THVD2442; symbol V2_Interface_RS485:THVD24x2 -> V2_Interface_RS485:THVD2442; Manufacturer (none) -> Texas Instruments; Mouser (none) -> 595-THVD2442DRCR; Product (none) -> THVD2442DRCR
Other:
- moved on the sheet: C1901, J1901, R1901, U1901

Commit message: Update library
Parts:
- C1901: Rating (none) -> 50V
Changed lines of the file:
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@@
 			)
 		)
-		(property "Description" "Power symbol creates a global label with name \"GND\" , ground"
+		(property "Description" ""
 			(at 167.64 64.77 0)
 			(effects
@@
 			)
 		)
-		(property "Description" "Power symbol creates a global label with name \"+5V\""
+		(property "Description" ""
 			(at 144.78 149.86 0)
 			(effects
@@
 			)
 		)
-		(property "Description" "Power symbol creates a global label with name \"GND\" , ground"
+		(property "Description" ""
 			(at 140.97 127 0)
 			(effects
@@
 			)
 		)
-		(property "Description" "Power symbol creates a global label with name \"+5V\""
+		(property "Description" ""
 			(at 140.97 132.08 0)
 			(effects
@@
 			)
 		)
-		(property "Description" "Power symbol creates a global label with name \"GND\" , ground"
+		(property "Description" ""
 			(at 147.32 97.79 0)
 			(effects
@@
 			)
 		)
-		(property "Description" "Power symbol creates a global label with name \"+5V\""
+		(property "Description" ""
 			(at 153.67 127 0)
 			(effects
@@
 			)
 		)
-		(property "Description" "Power symbol creates a global label with name \"+3V3\""
+		(property "Description" ""
 			(at 147.32 59.69 0)
 			(effects
@@
 			)
 		)
-		(property "Description" "Power symbol creates a global label with name \"GND\" , ground"
+		(property "Description" ""
 			(at 144.78 153.67 0)
 			(effects
@@
 			)
 		)
-		(property "Description" "Power symbol creates a global label with name \"GND\" , ground"
+		(property "Description" ""
 			(at 153.67 132.08 0)
 			(effects
@@
 			(effects
 				(font
+					(size 1.27 1.27)
+				)
+				(hide yes)
+			)
+		)
+		(property "Rating" "50V"
+			(at 167.64 85.09 0)
+			(effects
+				(font

Commit message: Update Library
Parts:
- C1901: symbol V2_Device:C_0603_0u1 -> V2_Capacitor:0603_0u1
- R1901: symbol V2_Device:R_0603_100R -> V2_Resistor:0603_100R
Changed lines of the file:
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@@
 	)
 	(symbol
-		(lib_id "V2_Device:R_0603_100R")
+		(lib_id "V2_Resistor:0603_100R")
 		(at 158.75 77.47 0)
 		(unit 1)
@@
 	)
 	(symbol
-		(lib_id "V2_Device:C_0603_0u1")
+		(lib_id "V2_Capacitor:0603_0u1")
 		(at 167.64 62.23 0)
 		(unit 1)

Commit message: Replace diode
Other:
- title: V2 Link -> V2 pulse
