File: hardware/pulse/LinkPlug.kicad_sch (KiCad schematic)
At the start: 4 parts, among them J1901 2x05_Horizontal, U1901 THVD2442

Commit message: Update
Parts:
- C1901: Id (none) -> Capacitor:${SYMBOL_NAME}
- J1901: Id (none) -> Header:${SYMBOL_NAME}
- R1901: Id (none) -> Resistor:${SYMBOL_NAME}
- U1901: Id (none) -> RS485:${SYMBOL_NAME}
Changed lines of the file:
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@@
+			)
+		)
+		(property "Id" "RS485:${SYMBOL_NAME}"
+			(at 147.32 114.3 0)
+			(hide yes)
+			(show_name no)
+			(do_not_autoplace no)
+			(effects
+				(font
+					(size 1.27 1.27)
+				)
 			)
 		)
@@
 			)
 		)
+		(property "Id" "Resistor:${SYMBOL_NAME}"
+			(at 158.75 91.44 0)
+			(hide yes)
+			(show_name no)
+			(do_not_autoplace no)
+			(effects
+				(font
+					(size 1.27 1.27)
+				)
+			)
+		)
 		(pin "1"
 		)
@@
 			)
 		)
+		(property "Id" "Header:${SYMBOL_NAME}"
+			(at 147.32 144.78 0)
+			(hide yes)
+			(show_name no)
+			(do_not_autoplace no)
+			(effects
+				(font
+					(size 1.27 1.27)
+				)
+			)
+		)
 		(pin "1"
 		)
@@
 			(hide yes)
 			(show_name no)
+			(do_not_autoplace no)
+			(effects
+				(font
+					(size 1.27 1.27)
+				)
+			)
+		)
+		(property "Id" "Capacitor:${SYMBOL_NAME}"
+			(at 167.64 77.47 0)
+			(hide yes)
+			(show_name no)

Commit message: Update
Parts:
- J1901: Rating (none) -> 1A
- U1901: Rating (none) -> 20Mbps
Other:
- company: Plug -> Versio Duo
Changed lines of the file:
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@@
 	(title_block
 		(title "V2 pulse")
-		(date "2026-03-30")
-		(rev "2026-03-30")
-		(company "Plug")
+		(date "2026-04-14")
+		(rev "2026-04-14")
+		(company "Versio Duo")
+		(comment 1 "Solenoid Controller")
 	)
 	(rectangle
@@
 		(in_pos_files yes)
 		(dnp no)
-		(property "Reference" "#PWR1902"
+		(property "Reference" "#PWR01909"
 			(at 167.64 71.12 0)
 			(hide yes)
@@
 			(project "pulse"
 				(path "/6c8448b4-b04d-47e1-934e-e40cbe27a7be/c6db2f80-f80f-4104-8ca1-02f0ab85cfea"
-					(reference "#PWR1902")
+					(reference "#PWR01909")
 					(unit 1)
 				)
@@
 		(in_pos_files yes)
 		(dnp no)
-		(property "Reference" "#FLG1902"
+		(property "Reference" "#FLG01902"
 			(at 146.685 153.67 0)
 			(hide yes)
@@
 			(project "pulse"
 				(path "/6c8448b4-b04d-47e1-934e-e40cbe27a7be/c6db2f80-f80f-4104-8ca1-02f0ab85cfea"
-					(reference "#FLG1902")
+					(reference "#FLG01902")
 					(unit 1)
 				)
@@
 		(in_pos_files yes)
 		(dnp no)
-		(property "Reference" "#FLG1901"
+		(property "Reference" "#FLG01901"
 			(at 146.685 149.86 0)
 			(hide yes)
@@
 			(project "pulse"
 				(path "/6c8448b4-b04d-47e1-934e-e40cbe27a7be/c6db2f80-f80f-4104-8ca1-02f0ab85cfea"
-					(reference "#FLG1901")
+					(reference "#FLG01901")
 					(unit 1)
 				)
@@
 			)
 		)
+		(property "Rating" "20Mbps"
+			(at 148.59 121.92 0)
+			(hide yes)
+			(show_name no)
+			(do_not_autoplace no)
+			(effects
+				(font
+					(size 1.27 1.27)
+				)
+			)
+		)
 		(pin "1"
 		)
@@
 			)
 		)
+		(property "Rating" "1A"
+			(at 147.32 160.02 0)
+			(hide yes)
+			(show_name no)
+			(do_not_autoplace no)
+			(effects
+				(font
+					(size 1.27 1.27)
+				)
+			)
+		)
 		(pin "1"
 		)
@@
 		(in_pos_files yes)
 		(dnp no)
-		(property "Reference" "#PWR1908"
+		(property "Reference" "#PWR01903"
 			(at 148.59 149.86 0)
 			(hide yes)
@@
 			(project "pulse"
 				(path "/6c8448b4-b04d-47e1-934e-e40cbe27a7be/c6db2f80-f80f-4104-8ca1-02f0ab85cfea"
-					(reference "#PWR1908")
+					(reference "#PWR01903")
 					(unit 1)
 				)
@@
 		(in_pos_files yes)
 		(dnp no)
-		(property "Reference" "#PWR1904"
+		(property "Reference" "#PWR01901"
 			(at 134.62 127 0)
 			(hide yes)
@@
 			(project "pulse"
 				(path "/6c8448b4-b04d-47e1-934e-e40cbe27a7be/c6db2f80-f80f-4104-8ca1-02f0ab85cfea"
-					(reference "#PWR1904")
+					(reference "#PWR01901")
 					(unit 1)
 				)
@@
 		(in_pos_files yes)
 		(dnp no)
-		(property "Reference" "#PWR1906"
+		(property "Reference" "#PWR01902"
 			(at 144.78 132.08 0)
 			(hide yes)
@@
 			(project "pulse"
 				(path "/6c8448b4-b04d-47e1-934e-e40cbe27a7be/c6db2f80-f80f-4104-8ca1-02f0ab85cfea"
-					(reference "#PWR1906")
+					(reference "#PWR01902")
 					(unit 1)
 				)
@@
 		(in_pos_files yes)
 		(dnp no)
-		(property "Reference" "#PWR1903"
+		(property "Reference" "#PWR01906"
 			(at 147.32 104.14 0)
 			(hide yes)
@@
 			(project "pulse"
 				(path "/6c8448b4-b04d-47e1-934e-e40cbe27a7be/c6db2f80-f80f-4104-8ca1-02f0ab85cfea"
-					(reference "#PWR1903")
+					(reference "#PWR01906")
 					(unit 1)
 				)
@@
 		(in_pos_files yes)
 		(dnp no)
-		(property "Reference" "#PWR1905"
+		(property "Reference" "#PWR01907"
 			(at 149.86 127 0)
 			(hide yes)
@@
 			(project "pulse"
 				(path "/6c8448b4-b04d-47e1-934e-e40cbe27a7be/c6db2f80-f80f-4104-8ca1-02f0ab85cfea"
-					(reference "#PWR1905")
+					(reference "#PWR01907")
 					(unit 1)
 				)
@@
 		(in_pos_files yes)
 		(dnp no)
-		(property "Reference" "#PWR1901"
+		(property "Reference" "#PWR01905"
 			(at 147.32 63.5 0)
 			(hide yes)
@@
 			(project "pulse"
 				(path "/6c8448b4-b04d-47e1-934e-e40cbe27a7be/c6db2f80-f80f-4104-8ca1-02f0ab85cfea"
-					(reference "#PWR1901")
+					(reference "#PWR01905")
 					(unit 1)
 				)
@@
 		(in_pos_files yes)
 		(dnp no)
-		(property "Reference" "#PWR1909"
+		(property "Reference" "#PWR01904"
 			(at 138.43 153.67 0)
 			(hide yes)
@@
 			(project "pulse"
 				(path "/6c8448b4-b04d-47e1-934e-e40cbe27a7be/c6db2f80-f80f-4104-8ca1-02f0ab85cfea"
-					(reference "#PWR1909")
+					(reference "#PWR01904")
 					(unit 1)
 				)
@@
 		(in_pos_files yes)
 		(dnp no)
-		(property "Reference" "#PWR1907"
+		(property "Reference" "#PWR01908"
 			(at 160.02 132.08 0)
 			(hide yes)
@@
 			(project "pulse"
 				(path "/6c8448b4-b04d-47e1-934e-e40cbe27a7be/c6db2f80-f80f-4104-8ca1-02f0ab85cfea"
-					(reference "#PWR1907")
+					(reference "#PWR01908")
 					(unit 1)
 				)

Commit message: Good Bye Imperial
Parts:
- C1901: footprint V2_Capacitor_SMD:C_0603 -> V2_Capacitor_SMD:C_1608; symbol V2_Capacitor:0603_0u1 -> V2_Capacitor:1608_0u1
- R1901: footprint V2_Resistor_SMD:R_0603 -> V2_Resistor_SMD:R_1608; symbol V2_Resistor:0603_100R -> V2_Resistor:1608_100R
Changed lines of the file:
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@@
 	)
 	(symbol
-		(lib_id "V2_Resistor:0603_100R")
+		(lib_id "V2_Resistor:1608_100R")
 		(at 158.75 77.47 0)
 		(unit 1)
@@
 			)
 		)
-		(property "Footprint" "V2_Resistor_SMD:R_0603"
+		(property "Footprint" "V2_Resistor_SMD:R_1608"
 			(at 158.75 93.218 0)
 			(hide yes)
@@
 	)
 	(symbol
-		(lib_id "V2_Capacitor:0603_0u1")
+		(lib_id "V2_Capacitor:1608_0u1")
 		(at 167.64 62.23 0)
 		(unit 1)
@@
 			)
 		)
-		(property "Footprint" "V2_Capacitor_SMD:C_0603"
+		(property "Footprint" "V2_Capacitor_SMD:C_1608"
 			(at 167.64 79.248 0)
 			(hide yes)
