File: hardware/pulse/LinkSocket.kicad_sch (KiCad schematic)
At the start: 4 parts, among them J2001 2x05_Horizontal, U2001 THVD2442

Commit message: Update
Parts:
- C2001: Id (none) -> Capacitor:${SYMBOL_NAME}
- J2001: Id (none) -> Header:${SYMBOL_NAME}
- R2001: Id (none) -> Resistor:${SYMBOL_NAME}
- U2001: Id (none) -> RS485:${SYMBOL_NAME}
Changed lines of the file:
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@@
+			)
+		)
+		(property "Id" "RS485:${SYMBOL_NAME}"
+			(at 151.13 119.38 0)
+			(hide yes)
+			(show_name no)
+			(do_not_autoplace no)
+			(effects
+				(font
+					(size 1.27 1.27)
+				)
 			)
 		)
@@
 			)
 		)
+		(property "Id" "Resistor:${SYMBOL_NAME}"
+			(at 162.56 96.52 0)
+			(hide yes)
+			(show_name no)
+			(do_not_autoplace no)
+			(effects
+				(font
+					(size 1.27 1.27)
+				)
+			)
+		)
 		(pin "1"
 		)
@@
 			)
 		)
+		(property "Id" "Header:${SYMBOL_NAME}"
+			(at 151.13 163.83 0)
+			(hide yes)
+			(show_name no)
+			(do_not_autoplace no)
+			(effects
+				(font
+					(size 1.27 1.27)
+				)
+			)
+		)
 		(pin "1"
 		)
@@
 			(hide yes)
 			(show_name no)
+			(do_not_autoplace no)
+			(effects
+				(font
+					(size 1.27 1.27)
+				)
+			)
+		)
+		(property "Id" "Capacitor:${SYMBOL_NAME}"
+			(at 172.72 82.55 0)
+			(hide yes)
+			(show_name no)

Commit message: Update
Parts:
- J2001: Rating (none) -> 1A
- U2001: Rating (none) -> 20Mbps
Other:
- company: Socket -> Versio Duo
Changed lines of the file:
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@@
 	(title_block
 		(title "V2 pulse")
-		(date "2026-03-30")
-		(rev "2026-03-30")
-		(company "Socket")
+		(date "2026-04-14")
+		(rev "2026-04-14")
+		(company "Versio Duo")
+		(comment 1 "Solenoid Controller")
 	)
 	(rectangle
@@
 		(in_pos_files yes)
 		(dnp no)
-		(property "Reference" "#PWR2001"
+		(property "Reference" "#PWR02003"
 			(at 151.13 68.58 0)
 			(hide yes)
@@
 			(project "pulse"
 				(path "/6c8448b4-b04d-47e1-934e-e40cbe27a7be/2a03ea79-269e-4abf-833c-000ba0ff13d7"
-					(reference "#PWR2001")
+					(reference "#PWR02003")
 					(unit 1)
 				)
@@
 			)
 		)
+		(property "Rating" "20Mbps"
+			(at 152.4 127 0)
+			(hide yes)
+			(show_name no)
+			(do_not_autoplace no)
+			(effects
+				(font
+					(size 1.27 1.27)
+				)
+			)
+		)
 		(pin "1"
 		)
@@
 		(in_pos_files yes)
 		(dnp no)
-		(property "Reference" "#PWR2004"
+		(property "Reference" "#PWR02001"
 			(at 138.43 146.05 0)
 			(hide yes)
@@
 			(project "pulse"
 				(path "/6c8448b4-b04d-47e1-934e-e40cbe27a7be/2a03ea79-269e-4abf-833c-000ba0ff13d7"
-					(reference "#PWR2004")
+					(reference "#PWR02001")
 					(unit 1)
 				)
@@
 		(in_pos_files yes)
 		(dnp no)
-		(property "Reference" "#PWR2003"
+		(property "Reference" "#PWR02004"
 			(at 151.13 109.22 0)
 			(hide yes)
@@
 			(project "pulse"
 				(path "/6c8448b4-b04d-47e1-934e-e40cbe27a7be/2a03ea79-269e-4abf-833c-000ba0ff13d7"
-					(reference "#PWR2003")
+					(reference "#PWR02004")
 					(unit 1)
 				)
@@
 		(in_pos_files yes)
 		(dnp no)
-		(property "Reference" "#PWR2002"
+		(property "Reference" "#PWR02007"
 			(at 172.72 76.2 0)
 			(hide yes)
@@
 			(project "pulse"
 				(path "/6c8448b4-b04d-47e1-934e-e40cbe27a7be/2a03ea79-269e-4abf-833c-000ba0ff13d7"
-					(reference "#PWR2002")
+					(reference "#PWR02007")
 					(unit 1)
 				)
@@
 		(in_pos_files yes)
 		(dnp no)
-		(property "Reference" "#PWR2007"
+		(property "Reference" "#PWR02006"
 			(at 163.83 151.13 0)
 			(hide yes)
@@
 			(project "pulse"
 				(path "/6c8448b4-b04d-47e1-934e-e40cbe27a7be/2a03ea79-269e-4abf-833c-000ba0ff13d7"
-					(reference "#PWR2007")
+					(reference "#PWR02006")
 					(unit 1)
 				)
@@
 			)
 		)
+		(property "Rating" "1A"
+			(at 151.13 179.07 0)
+			(hide yes)
+			(show_name no)
+			(do_not_autoplace no)
+			(effects
+				(font
+					(size 1.27 1.27)
+				)
+			)
+		)
 		(pin "1"
 		)
@@
 		(in_pos_files yes)
 		(dnp no)
-		(property "Reference" "#PWR2006"
+		(property "Reference" "#PWR02002"
 			(at 148.59 151.13 0)
 			(hide yes)
@@
 			(project "pulse"
 				(path "/6c8448b4-b04d-47e1-934e-e40cbe27a7be/2a03ea79-269e-4abf-833c-000ba0ff13d7"
-					(reference "#PWR2006")
+					(reference "#PWR02002")
 					(unit 1)
 				)
@@
 		(in_pos_files yes)
 		(dnp no)
-		(property "Reference" "#PWR2005"
+		(property "Reference" "#PWR02005"
 			(at 153.67 146.05 0)
 			(hide yes)
@@
 			(project "pulse"
 				(path "/6c8448b4-b04d-47e1-934e-e40cbe27a7be/2a03ea79-269e-4abf-833c-000ba0ff13d7"
-					(reference "#PWR2005")
+					(reference "#PWR02005")
 					(unit 1)
 				)

Commit message: Good Bye Imperial
Parts:
- C2001: footprint V2_Capacitor_SMD:C_0603 -> V2_Capacitor_SMD:C_1608; symbol V2_Capacitor:0603_0u1 -> V2_Capacitor:1608_0u1
- R2001: footprint V2_Resistor_SMD:R_0603 -> V2_Resistor_SMD:R_1608; symbol V2_Resistor:0603_100R -> V2_Resistor:1608_100R
Changed lines of the file:
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@@
 	)
 	(symbol
-		(lib_id "V2_Resistor:0603_100R")
+		(lib_id "V2_Resistor:1608_100R")
 		(at 162.56 82.55 0)
 		(unit 1)
@@
 			)
 		)
-		(property "Footprint" "V2_Resistor_SMD:R_0603"
+		(property "Footprint" "V2_Resistor_SMD:R_1608"
 			(at 162.56 98.298 0)
 			(hide yes)
@@
 	)
 	(symbol
-		(lib_id "V2_Capacitor:0603_0u1")
+		(lib_id "V2_Capacitor:1608_0u1")
 		(at 172.72 67.31 0)
 		(unit 1)
@@
 			)
 		)
-		(property "Footprint" "V2_Capacitor_SMD:C_0603"
+		(property "Footprint" "V2_Capacitor_SMD:C_1608"
 			(at 172.72 84.328 0)
 			(hide yes)
