File: hardware/pulse/PWMChannel.kicad_sch (KiCad schematic)
At the start: 6 parts, among them J201 WAGO 2065-100, J202 WAGO 2065-100, Q201 BSC010N04LS

Commit message: Replace diode
Other:
- title: Solenoid Channel -> V2 pulse

Commit message: Update
Parts:
- C201: Id (none) -> Capacitor:${SYMBOL_NAME}
- D201: Id (none) -> Diode:${SYMBOL_NAME}
- D202: Id (none) -> LED:${SYMBOL_NAME}
- J201, J202: Id (none) -> WAGO:${SYMBOL_NAME}
- Q201: Id (none) -> Mosfet:${SYMBOL_NAME}
Changed lines of the file:
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@@
+			)
+		)
+		(property "Id" "Diode:${SYMBOL_NAME}"
+			(at 127 93.98 0)
+			(hide yes)
+			(show_name no)
+			(do_not_autoplace no)
+			(effects
+				(font
+					(size 1.27 1.27)
+				)
 			)
 		)
@@
 			)
 		)
+		(property "Id" "Capacitor:${SYMBOL_NAME}"
+			(at 123.19 109.22 0)
+			(hide yes)
+			(show_name no)
+			(do_not_autoplace no)
+			(effects
+				(font
+					(size 1.27 1.27)
+				)
+			)
+		)
 		(pin "1"
 		)
@@
 			)
 		)
+		(property "Id" "Mosfet:${SYMBOL_NAME}"
+			(at 120.65 116.84 0)
+			(hide yes)
+			(show_name no)
+			(do_not_autoplace no)
+			(effects
+				(font
+					(size 1.27 1.27)
+				)
+			)
+		)
 		(pin "1"
 		)
@@
 		(in_bom no)
 		(on_board no)
-		(in_pos_files yes)
+		(in_pos_files no)
 		(dnp no)
 		(property "Reference" "#PWR201"
@@
 			)
 		)
+		(property "Id" "LED:${SYMBOL_NAME}"
+			(at 148.59 139.7 0)
+			(hide yes)
+			(show_name no)
+			(do_not_autoplace no)
+			(effects
+				(font
+					(size 1.27 1.27)
+				)
+			)
+		)
 		(pin "1"
 		)
@@
 			)
 		)
+		(property "Id" "WAGO:${SYMBOL_NAME}"
+			(at 165.1 97.79 0)
+			(hide yes)
+			(show_name no)
+			(do_not_autoplace no)
+			(effects
+				(font
+					(size 1.27 1.27)
+				)
+			)
+		)
 		(pin "1"
 		)
@@
 			(hide yes)
 			(show_name no)
+			(do_not_autoplace no)
+			(effects
+				(font
+					(size 1.27 1.27)
+				)
+			)
+		)
+		(property "Id" "WAGO:${SYMBOL_NAME}"
+			(at 165.1 102.87 0)
+			(hide yes)
+			(show_name no)

Commit message: Update
Parts:
- D202: Rating (none) -> 15mA
- J201, J202: Rating (none) -> 9A
- Q201: Id Mosfet:${SYMBOL_NAME} -> MOSFET:${SYMBOL_NAME}
Other:
- company: Power MOSFET + RGB LED -> Versio Duo

Commit message: Good Bye Imperial
Parts:
- C201: footprint V2_Capacitor_SMD:C_0603 -> V2_Capacitor_SMD:C_1608; symbol V2_Capacitor:0603_0u1 -> V2_Capacitor:1608_0u1
Changed lines of the file:
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@@
 	)
 	(symbol
-		(lib_id "V2_Capacitor:0603_0u1")
+		(lib_id "V2_Capacitor:1608_0u1")
 		(at 123.19 93.98 0)
 		(unit 1)
@@
 			)
 		)
-		(property "Footprint" "V2_Capacitor_SMD:C_0603"
+		(property "Footprint" "V2_Capacitor_SMD:C_1608"
 			(at 123.19 110.998 0)
 			(hide yes)
