File: hardware/pulse/Link-Plug.kicad_sch (KiCad schematic)
At the start: 4 parts, among them J2001 2x05_Horizontal

Commit message: Rename
Parts:
- removed C2001: 0u1, V2_Capacitor_SMD:C_1608, symbol V2_Capacitor:1608_0u1
- removed J2001: 2x05_Horizontal, V2_Connector_Header_1.27mm:PinHeader_2x05_P1.27mm_Horizontal, symbol V2_Connector_Header_1.27mm:2x05_Horizontal
- removed R2001: 100R, V2_Resistor_SMD:R_1608, symbol V2_Resistor:1608_100R
- removed U2001: (no value), V2_Package_SON:VSON-10-4-1EP_3x3mm_P0.5mm_EP1.65x2.4mm_ThermalVias, symbol V2_Interface_RS485:THVD24x2
- added C1901: 0u1, V2_Capacitor_SMD:C_1608, symbol V2_Capacitor:1608_0u1
- added J1901: 2x05_Horizontal, V2_Connector_Header_1.27mm:PinHeader_2x05_P1.27mm_Horizontal, symbol V2_Connector_Header_1.27mm:2x05_Horizontal
- added R1901: 100R, V2_Resistor_SMD:R_1608, symbol V2_Resistor:1608_100R
- added U1901: THVD2442, V2_Package_SON:VSON-10-4-1EP_3x3mm_P0.5mm_EP1.65x2.4mm_ThermalVias, symbol V2_Interface_RS485:THVD2442
Connections:
- net +3V3: now also C1901.1, U1901.10 (VCC)
- net +5V: now also J1901.4 (Pin_4), J1901.7 (Pin_7)
- net GND: now also C1901.2, J1901.3 (Pin_3), J1901.8 (Pin_8), U1901.11 (GND), U1901.5 (GND)
- net RX: now also U1901.1 (R)
- net RX-A: now also J1901.9 (Pin_9), R1901.1, U1901.9 (A)
- net RX-B: now also J1901.10 (Pin_10), R1901.2, U1901.8 (B)
- net RX-Enable: now also U1901.2 (RE)
- net TX: now also U1901.4 (D)
- net TX-Enable: now also U1901.3 (DE)
- net TX-Y: now also J1901.2 (Pin_2), U1901.6 (Y)
- net TX-Z: now also J1901.1 (Pin_1), U1901.7 (Z)
- new net USB+: J1901.5 (Pin_5)
- new net USB-: J1901.6 (Pin_6)
- no-connect marks 2 -> 0
Other:
- note added: "+5V from Plug"
- note added: "RS-422 3MHz"
- title: V2 pulse WAGO -> V2 pulse
