File: hardware/pulse-wago/pulse-wago.kicad_pcb (KiCad board)
At the start: 4 copper layers, 180 x 40 mm, 170 parts, among them J1001 WAGO 2601-1101, J1002 WAGO 2601-1101, J101 Cortex, J1101 WAGO 2601-1101, J1102 WAGO 2601-1101, J1201 WAGO 2601-1101, J1202 WAGO 2601-1101, J1301 WAGO 2601-1101, J1302 WAGO 2601-1101, J1401 WAGO 2601-1101, J1402 WAGO 2601-1101, J1501 WAGO 2601-1101, J1502 WAGO 2601-1101, J1601 WAGO 2601-1101, J1602 WAGO 2601-1101, J1701 WAGO 2601-1101, J1702 WAGO 2601-1101, J1801 WAGO 2065-100, J1802 WAGO 2065-100, J1901 2x05_Horizontal, J2001 2x05_Horizontal, J201 WAGO 2601-1101, J202 WAGO 2601-1101, J301 WAGO 2601-1101, J302 WAGO 2601-1101, J401 WAGO 2601-1101, J402 WAGO 2601-1101, J501 WAGO 2601-1101, J502 WAGO 2601-1101, J601 WAGO 2601-1101, J602 WAGO 2601-1101, J701 WAGO 2601-1101, J702 WAGO 2601-1101, J801 WAGO 2601-1101, J802 WAGO 2601-1101, J901 WAGO 2601-1101, J902 WAGO 2601-1101, Q1001 BSC010N04LS, Q1101 BSC010N04LS, Q1201 BSC010N04LS, Q1301 BSC010N04LS, Q1401 BSC010N04LS, Q1501 BSC010N04LS, Q1601 BSC010N04LS, Q1701 BSC010N04LS, Q201 BSC010N04LS, Q301 BSC010N04LS, Q401 BSC010N04LS, Q501 BSC010N04LS, Q601 BSC010N04LS, Q701 BSC010N04LS, Q801 BSC010N04LS, Q901 BSC010N04LS, SW101 SKSG, SW102 SKSG, U101 ATSAMD51J, U102 TPS78433QWDRBRQ1, U1801 BTT6010, Y101 32k768

Commit message: Replace Order_Number
Parts:
- H101, H103, H105, H107, H108: value MountingHole_2mm -> 2mm
- H102, H104, H106: value MountingHole_3mm -> 3mm
- INFO102: value Order_Number -> ~; footprint V2_Production:Order_Number -> V2_Production:Revision

Commit message: Replace diode
Parts:
- D1001, D1101, D1201, D1301, D1401, D1501, D1601, D1701, D201, D301, D401, D501, D601, D701, D801, D901: value S310FA -> PMEG6030AEXEX; footprint V2_Diode_SMD:D_SOD-123F -> V2_Diode_SMD:D_SOD-123HP
- moved D1001 0.75 mm to (164.8, 90.5)
- moved D1101 0.75 mm to (185.8, 90.5)
- moved D1201 0.75 mm to (178.8, 90.5)
- moved D1301 0.75 mm to (171.8, 90.5)
- moved D1401 0.75 mm to (192.8, 90.5)
- moved D1501 0.75 mm to (213.8, 90.5)
- moved D1601 0.75 mm to (206.8, 90.5)
- moved D1701 0.75 mm to (199.8, 90.5)
- moved D201 0.75 mm to (98.8, 90.5)
- moved D301 0.75 mm to (105.8, 90.5)
- moved D401 0.75 mm to (112.8, 90.5)
- moved D501 0.75 mm to (119.8, 90.5)
- moved D601 0.75 mm to (126.8, 90.5)
- moved D701 0.75 mm to (133.8, 90.5)
- moved D801 0.75 mm to (140.8, 90.5)
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Routing:
- net +28V: track 4.77 -> 4.27 mm, vias 139 -> 140
