File: hardware/pulse-wago/pulse-wago.kicad_pcb (KiCad board)
At the start: 4 copper layers, 180 x 40 mm, 170 parts, among them J1001 WAGO 2601-1101, J1002 WAGO 2601-1101, J101 Cortex, J1101 WAGO 2601-1101, J1102 WAGO 2601-1101, J1201 WAGO 2601-1101, J1202 WAGO 2601-1101, J1301 WAGO 2601-1101, J1302 WAGO 2601-1101, J1401 WAGO 2601-1101, J1402 WAGO 2601-1101, J1501 WAGO 2601-1101, J1502 WAGO 2601-1101, J1601 WAGO 2601-1101, J1602 WAGO 2601-1101, J1701 WAGO 2601-1101, J1702 WAGO 2601-1101, J1801 WAGO 2065-100, J1802 WAGO 2065-100, J1901 2x05_Horizontal, J2001 2x05_Horizontal, J201 WAGO 2601-1101, J202 WAGO 2601-1101, J301 WAGO 2601-1101, J302 WAGO 2601-1101, J401 WAGO 2601-1101, J402 WAGO 2601-1101, J501 WAGO 2601-1101, J502 WAGO 2601-1101, J601 WAGO 2601-1101, J602 WAGO 2601-1101, J701 WAGO 2601-1101, J702 WAGO 2601-1101, J801 WAGO 2601-1101, J802 WAGO 2601-1101, J901 WAGO 2601-1101, J902 WAGO 2601-1101, Q1001 BSC010N04LS, Q1101 BSC010N04LS, Q1201 BSC010N04LS, Q1301 BSC010N04LS, Q1401 BSC010N04LS, Q1501 BSC010N04LS, Q1601 BSC010N04LS, Q1701 BSC010N04LS, Q201 BSC010N04LS, Q301 BSC010N04LS, Q401 BSC010N04LS, Q501 BSC010N04LS, Q601 BSC010N04LS, Q701 BSC010N04LS, Q801 BSC010N04LS, Q901 BSC010N04LS, SW101 SKSG, SW102 SKSG, U101 ATSAMD51J, U102 TPS78433QWDRBRQ1, U1801 BTT6010, Y101 32k768

Commit message: Replace diode
Parts:
- D1801: value RB501SM -> PMEG2010EPK; footprint V2_Diode_SMD:D_SOD-523 -> V2_Diode_SMD:D_SOD-1608

Commit message: Update
Parts:
- renumbered C107 to C101, C108 to C102, C109 to C103, C101 to C104, C110 to C105, C102 to C106, C103 to C107, C104 to C108, C105 to C109, C106 to C110, C1807 to C1801, C1801 to C1802, C1802 to C1803, C1803 to C1807, D102 to D101, D101 to D102, H103 to H102, H105 to H103, H107 to H104, H108 to H105, H102 to H106, H104 to H107, H106 to H108, ICON104 to ICON101, ICON105 to ICON102, ICON101 to ICON103, ICON102 to ICON104, ICON103 to ICON105, R102 to R101, R101 to R102, R1804 to R1801, R1808 to R1802, R1807 to R1803, R1809 to R1804, R1810 to R1805, R1801 to R1807, R1803 to R1808, R1805 to R1809, R1802 to R1810, SW102 to SW101, SW101 to SW102, U102 to U101, U101 to U102
