File: hardware/pulse-wago/LinkPlug.kicad_sch (KiCad schematic)
At the start: 4 parts, among them J1901 2x05_Horizontal, U1901 THVD24x2

Commit message: Update library
Parts:
- C1901: footprint Capacitor_SMD:C_0603_1608Metric -> V2_Capacitor_SMD:C_0603; symbol Device:C_Small -> V2_Device:C_0603_0u1; Manufacturer (none) -> TDK; Mouser (none) -> 810-CGA3E2X7R1H104MA; Product (none) -> CGA3E2X7R1H104M080AA; Rating (none) -> 50V
- J1901: Manufacturer (none) -> Amphenol FCI; Mouser (none) -> 649-200211120001T4LF; Product (none) -> 20021112-00010T4LF
- R1901: footprint Resistor_SMD:R_0603_1608Metric -> V2_Resistor_SMD:R_0603; symbol Device:R_Small -> V2_Device:R_0603_100R; Manufacturer (none) -> Vishay; Mouser (none) -> 71-CRCW0603100RFKEAH; Product (none) -> CRCW0603100RFKEAHP; Rating (none) -> 330mW
- U1901: value THVD24x2 -> (none)
Other:
- moved on the sheet: C1901, J1901, R1901, U1901

Commit message: Update Library
Parts:
- C1901: symbol V2_Device:C_0603_0u1 -> V2_Capacitor:0603_0u1
- R1901: symbol V2_Device:R_0603_100R -> V2_Resistor:0603_100R
Changed lines of the file:
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@@
 		(on_board yes)
 		(dnp no)
-		(property "Reference" "#PWR01902"
+		(property "Reference" "#PWR1902"
 			(at 176.53 80.01 0)
 			(effects
@@
 			(project "pulse"
 				(path "/6c8448b4-b04d-47e1-934e-e40cbe27a7be/c6db2f80-f80f-4104-8ca1-02f0ab85cfea"
-					(reference "#PWR01902")
+					(reference "#PWR1902")
 					(unit 1)
 				)
@@
 		(on_board yes)
 		(dnp no)
-		(property "Reference" "#FLG01902"
+		(property "Reference" "#FLG1902"
 			(at 160.02 46.355 0)
 			(effects
@@
 			(project "pulse"
 				(path "/6c8448b4-b04d-47e1-934e-e40cbe27a7be/c6db2f80-f80f-4104-8ca1-02f0ab85cfea"
-					(reference "#FLG01902")
+					(reference "#FLG1902")
 					(unit 1)
 				)
@@
 		(on_board yes)
 		(dnp no)
-		(property "Reference" "#FLG01901"
+		(property "Reference" "#FLG1901"
 			(at 160.02 42.545 0)
 			(effects
@@
 			(project "pulse"
 				(path "/6c8448b4-b04d-47e1-934e-e40cbe27a7be/c6db2f80-f80f-4104-8ca1-02f0ab85cfea"
-					(reference "#FLG01901")
+					(reference "#FLG1901")
 					(unit 1)
 				)
@@
 	)
 	(symbol
-		(lib_id "V2_Device:R_0603_100R")
+		(lib_id "V2_Resistor:0603_100R")
 		(at 168.91 86.36 0)
 		(unit 1)
@@
 		(on_board yes)
 		(dnp no)
-		(property "Reference" "#PWR01908"
+		(property "Reference" "#PWR1908"
 			(at 156.21 44.45 0)
 			(effects
@@
 			(project "pulse"
 				(path "/6c8448b4-b04d-47e1-934e-e40cbe27a7be/c6db2f80-f80f-4104-8ca1-02f0ab85cfea"
-					(reference "#PWR01908")
+					(reference "#PWR1908")
 					(unit 1)
 				)
@@
 		(on_board yes)
 		(dnp no)
-		(property "Reference" "#PWR01904"
+		(property "Reference" "#PWR1904"
 			(at 143.51 142.24 0)
 			(effects
@@
 			(project "pulse"
 				(path "/6c8448b4-b04d-47e1-934e-e40cbe27a7be/c6db2f80-f80f-4104-8ca1-02f0ab85cfea"
-					(reference "#PWR01904")
+					(reference "#PWR1904")
 					(unit 1)
 				)
@@
 		(on_board yes)
 		(dnp no)
-		(property "Reference" "#PWR01906"
+		(property "Reference" "#PWR1906"
 			(at 153.67 147.32 0)
 			(effects
@@
 			(project "pulse"
 				(path "/6c8448b4-b04d-47e1-934e-e40cbe27a7be/c6db2f80-f80f-4104-8ca1-02f0ab85cfea"
-					(reference "#PWR01906")
+					(reference "#PWR1906")
 					(unit 1)
 				)
@@
 		(on_board yes)
 		(dnp no)
-		(property "Reference" "#PWR01903"
+		(property "Reference" "#PWR1903"
 			(at 156.21 113.03 0)
 			(effects
@@
 			(project "pulse"
 				(path "/6c8448b4-b04d-47e1-934e-e40cbe27a7be/c6db2f80-f80f-4104-8ca1-02f0ab85cfea"
-					(reference "#PWR01903")
+					(reference "#PWR1903")
 					(unit 1)
 				)
@@
 		(on_board yes)
 		(dnp no)
-		(property "Reference" "#PWR01905"
+		(property "Reference" "#PWR1905"
 			(at 158.75 142.24 0)
 			(effects
@@
 			(project "pulse"
 				(path "/6c8448b4-b04d-47e1-934e-e40cbe27a7be/c6db2f80-f80f-4104-8ca1-02f0ab85cfea"
-					(reference "#PWR01905")
+					(reference "#PWR1905")
 					(unit 1)
 				)
@@
 		(on_board yes)
 		(dnp no)
-		(property "Reference" "#PWR01901"
+		(property "Reference" "#PWR1901"
 			(at 156.21 72.39 0)
 			(effects
@@
 			(project "pulse"
 				(path "/6c8448b4-b04d-47e1-934e-e40cbe27a7be/c6db2f80-f80f-4104-8ca1-02f0ab85cfea"
-					(reference "#PWR01901")
+					(reference "#PWR1901")
 					(unit 1)
 				)
@@
 		(on_board yes)
 		(dnp no)
-		(property "Reference" "#PWR01909"
+		(property "Reference" "#PWR1909"
 			(at 166.37 48.26 0)
 			(effects
@@
 			(project "pulse"
 				(path "/6c8448b4-b04d-47e1-934e-e40cbe27a7be/c6db2f80-f80f-4104-8ca1-02f0ab85cfea"
-					(reference "#PWR01909")
+					(reference "#PWR1909")
 					(unit 1)
 				)
@@
 		(on_board yes)
 		(dnp no)
-		(property "Reference" "#PWR01907"
+		(property "Reference" "#PWR1907"
 			(at 168.91 147.32 0)
 			(effects
@@
 			(project "pulse"
 				(path "/6c8448b4-b04d-47e1-934e-e40cbe27a7be/c6db2f80-f80f-4104-8ca1-02f0ab85cfea"
-					(reference "#PWR01907")
-					(unit 1)
-				)
-			)
-		)
-	)
-	(symbol
-		(lib_id "V2_Device:C_0603_0u1")
+					(reference "#PWR1907")
+					(unit 1)
+				)
+			)
+		)
+	)
+	(symbol
+		(lib_id "V2_Capacitor:0603_0u1")
 		(at 176.53 71.12 0)
 		(unit 1)

Commit message: Update ESD suppressor
Parts:
- U1901: value (none) -> ~
Changed lines of the file:
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@@
 			)
 		)
-		(property "Value" ""
+		(property "Value" "~"
 			(at 158.3533 76.2 0)
 			(effects

Commit message: Replace diode
Parts:
- U1901: value ~ -> (none)
Other:
- title: V2 Link -> V2 pulse WAGO

Commit message: Update
Parts:
- C1901: Id (none) -> Capacitor:${SYMBOL_NAME}
- J1901: Id (none) -> Header:${SYMBOL_NAME}; Rating (none) -> 1A
- R1901: Id (none) -> Resistor:${SYMBOL_NAME}
- U1901: Id (none) -> RS485:${SYMBOL_NAME}
Other:
- company: Plug -> Versio Duo
Changed lines of the file:
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@@
 	(title_block
 		(title "V2 pulse WAGO")
-		(date "2026-03-30")
-		(rev "2026-03-30")
-		(company "Plug")
+		(date "2026-04-14")
+		(rev "2026-04-14")
+		(company "Versio Duo")
+		(comment 1 "Solenoid Controller")
 	)
 	(rectangle
@@
 		(in_pos_files yes)
 		(dnp no)
-		(property "Reference" "#PWR1902"
+		(property "Reference" "#PWR01909"
 			(at 176.53 80.01 0)
 			(hide yes)
@@
 			(project "pulse-wago"
 				(path "/6c8448b4-b04d-47e1-934e-e40cbe27a7be/c6db2f80-f80f-4104-8ca1-02f0ab85cfea"
-					(reference "#PWR1902")
+					(reference "#PWR01909")
 					(unit 1)
 				)
@@
 		(in_pos_files yes)
 		(dnp no)
-		(property "Reference" "#FLG1902"
+		(property "Reference" "#FLG01902"
 			(at 160.02 46.355 0)
 			(hide yes)
@@
 			(project "pulse-wago"
 				(path "/6c8448b4-b04d-47e1-934e-e40cbe27a7be/c6db2f80-f80f-4104-8ca1-02f0ab85cfea"
-					(reference "#FLG1902")
+					(reference "#FLG01902")
 					(unit 1)
 				)
@@
 		(in_pos_files yes)
 		(dnp no)
-		(property "Reference" "#FLG1901"
+		(property "Reference" "#FLG01901"
 			(at 160.02 42.545 0)
 			(hide yes)
@@
 			(project "pulse-wago"
 				(path "/6c8448b4-b04d-47e1-934e-e40cbe27a7be/c6db2f80-f80f-4104-8ca1-02f0ab85cfea"
-					(reference "#FLG1901")
+					(reference "#FLG01901")
 					(unit 1)
 				)
@@
 			)
 		)
+		(property "Id" "RS485:${SYMBOL_NAME}"
+			(at 156.21 123.19 0)
+			(hide yes)
+			(show_name no)
+			(do_not_autoplace no)
+			(effects
+				(font
+					(size 1.27 1.27)
+				)
+			)
+		)
 		(pin "1"
 		)
@@
 			)
 		)
+		(property "Id" "Resistor:${SYMBOL_NAME}"
+			(at 168.91 100.33 0)
+			(hide yes)
+			(show_name no)
+			(do_not_autoplace no)
+			(effects
+				(font
+					(size 1.27 1.27)
+				)
+			)
+		)
 		(pin "1"
 		)
@@
 			)
 		)
+		(property "Id" "Header:${SYMBOL_NAME}"
+			(at 156.21 160.02 0)
+			(hide yes)
+			(show_name no)
+			(do_not_autoplace no)
+			(effects
+				(font
+					(size 1.27 1.27)
+				)
+			)
+		)
+		(property "Rating" "1A"
+			(at 156.21 175.26 0)
+			(hide yes)
+			(show_name no)
+			(do_not_autoplace no)
+			(effects
+				(font
+					(size 1.27 1.27)
+				)
+			)
+		)
 		(pin "1"
 		)
@@
 		(in_pos_files yes)
 		(dnp no)
-		(property "Reference" "#PWR1908"
+		(property "Reference" "#PWR01905"
 			(at 156.21 44.45 0)
 			(hide yes)
@@
 			(project "pulse-wago"
 				(path "/6c8448b4-b04d-47e1-934e-e40cbe27a7be/c6db2f80-f80f-4104-8ca1-02f0ab85cfea"
-					(reference "#PWR1908")
+					(reference "#PWR01905")
 					(unit 1)
 				)
@@
 		(in_pos_files yes)
 		(dnp no)
-		(property "Reference" "#PWR1904"
+		(property "Reference" "#PWR01901"
 			(at 143.51 142.24 0)
 			(hide yes)
@@
 			(project "pulse-wago"
 				(path "/6c8448b4-b04d-47e1-934e-e40cbe27a7be/c6db2f80-f80f-4104-8ca1-02f0ab85cfea"
-					(reference "#PWR1904")
+					(reference "#PWR01901")
 					(unit 1)
 				)
@@
 		(in_pos_files yes)
 		(dnp no)
-		(property "Reference" "#PWR1906"
+		(property "Reference" "#PWR01902"
 			(at 153.67 147.32 0)
 			(hide yes)
@@
 			(project "pulse-wago"
 				(path "/6c8448b4-b04d-47e1-934e-e40cbe27a7be/c6db2f80-f80f-4104-8ca1-02f0ab85cfea"
-					(reference "#PWR1906")
+					(reference "#PWR01902")
 					(unit 1)
 				)
@@
 		(in_pos_files yes)
 		(dnp no)
-		(property "Reference" "#PWR1903"
+		(property "Reference" "#PWR01904"
 			(at 156.21 113.03 0)
 			(hide yes)
@@
 			(project "pulse-wago"
 				(path "/6c8448b4-b04d-47e1-934e-e40cbe27a7be/c6db2f80-f80f-4104-8ca1-02f0ab85cfea"
-					(reference "#PWR1903")
+					(reference "#PWR01904")
 					(unit 1)
 				)
@@
 		(in_pos_files yes)
 		(dnp no)
-		(property "Reference" "#PWR1905"
+		(property "Reference" "#PWR01907"
 			(at 158.75 142.24 0)
 			(hide yes)
@@
 			(project "pulse-wago"
 				(path "/6c8448b4-b04d-47e1-934e-e40cbe27a7be/c6db2f80-f80f-4104-8ca1-02f0ab85cfea"
-					(reference "#PWR1905")
+					(reference "#PWR01907")
 					(unit 1)
 				)
@@
 		(in_pos_files yes)
 		(dnp no)
-		(property "Reference" "#PWR1901"
+		(property "Reference" "#PWR01903"
 			(at 156.21 72.39 0)
 			(hide yes)
@@
 			(project "pulse-wago"
 				(path "/6c8448b4-b04d-47e1-934e-e40cbe27a7be/c6db2f80-f80f-4104-8ca1-02f0ab85cfea"
-					(reference "#PWR1901")
+					(reference "#PWR01903")
 					(unit 1)
 				)
@@
 		(in_pos_files yes)
 		(dnp no)
-		(property "Reference" "#PWR1909"
+		(property "Reference" "#PWR01906"
 			(at 166.37 48.26 0)
 			(hide yes)
@@
 			(project "pulse-wago"
 				(path "/6c8448b4-b04d-47e1-934e-e40cbe27a7be/c6db2f80-f80f-4104-8ca1-02f0ab85cfea"
-					(reference "#PWR1909")
+					(reference "#PWR01906")
 					(unit 1)
 				)
@@
 		(in_pos_files yes)
 		(dnp no)
-		(property "Reference" "#PWR1907"
+		(property "Reference" "#PWR01908"
 			(at 168.91 147.32 0)
 			(hide yes)
@@
 			(project "pulse-wago"
 				(path "/6c8448b4-b04d-47e1-934e-e40cbe27a7be/c6db2f80-f80f-4104-8ca1-02f0ab85cfea"
-					(reference "#PWR1907")
+					(reference "#PWR01908")
 					(unit 1)
 				)
@@
 			(hide yes)
 			(show_name no)
+			(do_not_autoplace no)
+			(effects
+				(font
+					(size 1.27 1.27)
+				)
+			)
+		)
+		(property "Id" "Capacitor:${SYMBOL_NAME}"
+			(at 176.53 86.36 0)
+			(hide yes)
+			(show_name no)

Commit message: Good Bye Imperial
Parts:
- C1901: footprint V2_Capacitor_SMD:C_0603 -> V2_Capacitor_SMD:C_1608; symbol V2_Capacitor:0603_0u1 -> V2_Capacitor:1608_0u1
- R1901: footprint V2_Resistor_SMD:R_0603 -> V2_Resistor_SMD:R_1608; symbol V2_Resistor:0603_100R -> V2_Resistor:1608_100R
Changed lines of the file:
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@@
 	)
 	(symbol
-		(lib_id "V2_Resistor:0603_100R")
+		(lib_id "V2_Resistor:1608_100R")
 		(at 168.91 86.36 0)
 		(unit 1)
@@
 			)
 		)
-		(property "Footprint" "V2_Resistor_SMD:R_0603"
+		(property "Footprint" "V2_Resistor_SMD:R_1608"
 			(at 168.91 102.108 0)
 			(hide yes)
@@
 	)
 	(symbol
-		(lib_id "V2_Capacitor:0603_0u1")
+		(lib_id "V2_Capacitor:1608_0u1")
 		(at 176.53 71.12 0)
 		(unit 1)
@@
 			)
 		)
-		(property "Footprint" "V2_Capacitor_SMD:C_0603"
+		(property "Footprint" "V2_Capacitor_SMD:C_1608"
 			(at 176.53 88.138 0)
 			(hide yes)
