File: hardware/pulse-wago/LinkSocket.kicad_sch (KiCad schematic)
At the start: 4 parts, among them J2001 2x05_Horizontal, U2001 THVD24x2

Commit message: Update library
Parts:
- C2001: footprint Capacitor_SMD:C_0603_1608Metric -> V2_Capacitor_SMD:C_0603; symbol Device:C_Small -> V2_Device:C_0603_0u1; Manufacturer (none) -> TDK; Mouser (none) -> 810-CGA3E2X7R1H104MA; Product (none) -> CGA3E2X7R1H104M080AA; Rating (none) -> 50V
- J2001: Manufacturer (none) -> Amphenol FCI; Mouser (none) -> 649-200211120001T4LF; Product (none) -> 20021112-00010T4LF
- R2001: footprint Resistor_SMD:R_0603_1608Metric -> V2_Resistor_SMD:R_0603; symbol Device:R_Small -> V2_Device:R_0603_100R; Manufacturer (none) -> Vishay; Mouser (none) -> 71-CRCW0603100RFKEAH; Product (none) -> CRCW0603100RFKEAHP; Rating (none) -> 330mW
- U2001: value THVD24x2 -> (none)
Other:
- moved on the sheet: C2001, J2001, R2001, U2001

Commit message: Update Library
Parts:
- C2001: symbol V2_Device:C_0603_0u1 -> V2_Capacitor:0603_0u1
- R2001: symbol V2_Device:R_0603_100R -> V2_Resistor:0603_100R
Changed lines of the file:
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@@
 		(on_board yes)
 		(dnp no)
-		(property "Reference" "#PWR02001"
+		(property "Reference" "#PWR2001"
 			(at 151.13 69.85 0)
 			(effects
@@
 			(project "pulse"
 				(path "/6c8448b4-b04d-47e1-934e-e40cbe27a7be/2a03ea79-269e-4abf-833c-000ba0ff13d7"
-					(reference "#PWR02001")
+					(reference "#PWR2001")
 					(unit 1)
 				)
@@
 		(on_board yes)
 		(dnp no)
-		(property "Reference" "#PWR02004"
+		(property "Reference" "#PWR2004"
 			(at 138.43 139.7 0)
 			(effects
@@
 			(project "pulse"
 				(path "/6c8448b4-b04d-47e1-934e-e40cbe27a7be/2a03ea79-269e-4abf-833c-000ba0ff13d7"
-					(reference "#PWR02004")
+					(reference "#PWR2004")
 					(unit 1)
 				)
@@
 		(on_board yes)
 		(dnp no)
-		(property "Reference" "#PWR02003"
+		(property "Reference" "#PWR2003"
 			(at 151.13 110.49 0)
 			(effects
@@
 			(project "pulse"
 				(path "/6c8448b4-b04d-47e1-934e-e40cbe27a7be/2a03ea79-269e-4abf-833c-000ba0ff13d7"
-					(reference "#PWR02003")
+					(reference "#PWR2003")
 					(unit 1)
 				)
@@
 		(on_board yes)
 		(dnp no)
-		(property "Reference" "#PWR02002"
+		(property "Reference" "#PWR2002"
 			(at 172.72 77.47 0)
 			(effects
@@
 			(project "pulse"
 				(path "/6c8448b4-b04d-47e1-934e-e40cbe27a7be/2a03ea79-269e-4abf-833c-000ba0ff13d7"
-					(reference "#PWR02002")
-					(unit 1)
-				)
-			)
-		)
-	)
-	(symbol
-		(lib_id "V2_Device:R_0603_100R")
+					(reference "#PWR2002")
+					(unit 1)
+				)
+			)
+		)
+	)
+	(symbol
+		(lib_id "V2_Resistor:0603_100R")
 		(at 163.83 83.82 0)
 		(unit 1)
@@
 		(on_board yes)
 		(dnp no)
-		(property "Reference" "#PWR02007"
+		(property "Reference" "#PWR2007"
 			(at 163.83 144.78 0)
 			(effects
@@
 			(project "pulse"
 				(path "/6c8448b4-b04d-47e1-934e-e40cbe27a7be/2a03ea79-269e-4abf-833c-000ba0ff13d7"
-					(reference "#PWR02007")
+					(reference "#PWR2007")
 					(unit 1)
 				)
@@
 	)
 	(symbol
-		(lib_id "V2_Device:C_0603_0u1")
+		(lib_id "V2_Capacitor:0603_0u1")
 		(at 172.72 68.58 0)
 		(unit 1)
@@
 		(on_board yes)
 		(dnp no)
-		(property "Reference" "#PWR02006"
+		(property "Reference" "#PWR2006"
 			(at 148.59 144.78 0)
 			(effects
@@
 			(project "pulse"
 				(path "/6c8448b4-b04d-47e1-934e-e40cbe27a7be/2a03ea79-269e-4abf-833c-000ba0ff13d7"
-					(reference "#PWR02006")
+					(reference "#PWR2006")
 					(unit 1)
 				)
@@
 		(on_board yes)
 		(dnp no)
-		(property "Reference" "#PWR02005"
+		(property "Reference" "#PWR2005"
 			(at 153.67 139.7 0)
 			(effects
@@
 			(project "pulse"
 				(path "/6c8448b4-b04d-47e1-934e-e40cbe27a7be/2a03ea79-269e-4abf-833c-000ba0ff13d7"
-					(reference "#PWR02005")
-					(unit 1)
-				)
+					(reference "#PWR2005")
+					(unit 1)
+				)

Commit message: Update ESD suppressor
Parts:
- U2001: value (none) -> ~
Changed lines of the file:
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@@
 			)
 		)
-		(property "Value" ""
+		(property "Value" "~"
 			(at 153.67 73.66 0)
 			(effects

Commit message: Replace diode
Parts:
- U2001: value ~ -> (none)
Other:
- title: V2 Link -> V2 pulse WAGO

Commit message: Update
Parts:
- C2001: Id (none) -> Capacitor:${SYMBOL_NAME}
- J2001: Id (none) -> Header:${SYMBOL_NAME}; Rating (none) -> 1A
- R2001: Id (none) -> Resistor:${SYMBOL_NAME}
- U2001: Id (none) -> RS485:${SYMBOL_NAME}
Other:
- company: Socket -> Versio Duo
Changed lines of the file:
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@@
 	(title_block
 		(title "V2 pulse WAGO")
-		(date "2026-03-30")
-		(rev "2026-03-30")
-		(company "Socket")
+		(date "2026-04-14")
+		(rev "2026-04-14")
+		(company "Versio Duo")
+		(comment 1 "Solenoid Controller")
 	)
 	(rectangle
@@
 		(in_pos_files yes)
 		(dnp no)
-		(property "Reference" "#PWR2001"
+		(property "Reference" "#PWR02003"
 			(at 151.13 69.85 0)
 			(hide yes)
@@
 			(project "pulse-wago"
 				(path "/6c8448b4-b04d-47e1-934e-e40cbe27a7be/2a03ea79-269e-4abf-833c-000ba0ff13d7"
-					(reference "#PWR2001")
+					(reference "#PWR02003")
 					(unit 1)
 				)
@@
 			)
 		)
+		(property "Id" "RS485:${SYMBOL_NAME}"
+			(at 151.13 120.65 0)
+			(hide yes)
+			(show_name no)
+			(do_not_autoplace no)
+			(effects
+				(font
+					(size 1.27 1.27)
+				)
+			)
+		)
 		(pin "1"
 		)
@@
 		(in_pos_files yes)
 		(dnp no)
-		(property "Reference" "#PWR2004"
+		(property "Reference" "#PWR02001"
 			(at 138.43 139.7 0)
 			(hide yes)
@@
 			(project "pulse-wago"
 				(path "/6c8448b4-b04d-47e1-934e-e40cbe27a7be/2a03ea79-269e-4abf-833c-000ba0ff13d7"
-					(reference "#PWR2004")
+					(reference "#PWR02001")
 					(unit 1)
 				)
@@
 		(in_pos_files yes)
 		(dnp no)
-		(property "Reference" "#PWR2003"
+		(property "Reference" "#PWR02004"
 			(at 151.13 110.49 0)
 			(hide yes)
@@
 			(project "pulse-wago"
 				(path "/6c8448b4-b04d-47e1-934e-e40cbe27a7be/2a03ea79-269e-4abf-833c-000ba0ff13d7"
-					(reference "#PWR2003")
+					(reference "#PWR02004")
 					(unit 1)
 				)
@@
 		(in_pos_files yes)
 		(dnp no)
-		(property "Reference" "#PWR2002"
+		(property "Reference" "#PWR02007"
 			(at 172.72 77.47 0)
 			(hide yes)
@@
 			(project "pulse-wago"
 				(path "/6c8448b4-b04d-47e1-934e-e40cbe27a7be/2a03ea79-269e-4abf-833c-000ba0ff13d7"
-					(reference "#PWR2002")
+					(reference "#PWR02007")
 					(unit 1)
 				)
@@
 			)
 		)
+		(property "Id" "Resistor:${SYMBOL_NAME}"
+			(at 163.83 97.79 0)
+			(hide yes)
+			(show_name no)
+			(do_not_autoplace no)
+			(effects
+				(font
+					(size 1.27 1.27)
+				)
+			)
+		)
 		(pin "1"
 		)
@@
 		(in_pos_files yes)
 		(dnp no)
-		(property "Reference" "#PWR2007"
+		(property "Reference" "#PWR02006"
 			(at 163.83 144.78 0)
 			(hide yes)
@@
 			(project "pulse-wago"
 				(path "/6c8448b4-b04d-47e1-934e-e40cbe27a7be/2a03ea79-269e-4abf-833c-000ba0ff13d7"
-					(reference "#PWR2007")
+					(reference "#PWR02006")
 					(unit 1)
 				)
@@
 			)
 		)
+		(property "Id" "Header:${SYMBOL_NAME}"
+			(at 151.13 157.48 0)
+			(hide yes)
+			(show_name no)
+			(do_not_autoplace no)
+			(effects
+				(font
+					(size 1.27 1.27)
+				)
+			)
+		)
+		(property "Rating" "1A"
+			(at 151.13 172.72 0)
+			(hide yes)
+			(show_name no)
+			(do_not_autoplace no)
+			(effects
+				(font
+					(size 1.27 1.27)
+				)
+			)
+		)
 		(pin "1"
 		)
@@
 			)
 		)
+		(property "Id" "Capacitor:${SYMBOL_NAME}"
+			(at 172.72 83.82 0)
+			(hide yes)
+			(show_name no)
+			(do_not_autoplace no)
+			(effects
+				(font
+					(size 1.27 1.27)
+				)
+			)
+		)
 		(pin "1"
 		)
@@
 		(in_pos_files yes)
 		(dnp no)
-		(property "Reference" "#PWR2006"
+		(property "Reference" "#PWR02002"
 			(at 148.59 144.78 0)
 			(hide yes)
@@
 			(project "pulse-wago"
 				(path "/6c8448b4-b04d-47e1-934e-e40cbe27a7be/2a03ea79-269e-4abf-833c-000ba0ff13d7"
-					(reference "#PWR2006")
+					(reference "#PWR02002")
 					(unit 1)
 				)
@@
 		(in_pos_files yes)
 		(dnp no)
-		(property "Reference" "#PWR2005"
+		(property "Reference" "#PWR02005"
 			(at 153.67 139.7 0)
 			(hide yes)
@@
 			(project "pulse-wago"
 				(path "/6c8448b4-b04d-47e1-934e-e40cbe27a7be/2a03ea79-269e-4abf-833c-000ba0ff13d7"
-					(reference "#PWR2005")
+					(reference "#PWR02005")
 					(unit 1)
 				)

Commit message: Good Bye Imperial
Parts:
- C2001: footprint V2_Capacitor_SMD:C_0603 -> V2_Capacitor_SMD:C_1608; symbol V2_Capacitor:0603_0u1 -> V2_Capacitor:1608_0u1
- R2001: footprint V2_Resistor_SMD:R_0603 -> V2_Resistor_SMD:R_1608; symbol V2_Resistor:0603_100R -> V2_Resistor:1608_100R
Changed lines of the file:
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@@
 	)
 	(symbol
-		(lib_id "V2_Resistor:0603_100R")
+		(lib_id "V2_Resistor:1608_100R")
 		(at 163.83 83.82 0)
 		(unit 1)
@@
 			)
 		)
-		(property "Footprint" "V2_Resistor_SMD:R_0603"
+		(property "Footprint" "V2_Resistor_SMD:R_1608"
 			(at 163.83 99.568 0)
 			(hide yes)
@@
 	)
 	(symbol
-		(lib_id "V2_Capacitor:0603_0u1")
+		(lib_id "V2_Capacitor:1608_0u1")
 		(at 172.72 68.58 0)
 		(unit 1)
@@
 			)
 		)
-		(property "Footprint" "V2_Capacitor_SMD:C_0603"
+		(property "Footprint" "V2_Capacitor_SMD:C_1608"
 			(at 172.72 85.598 0)
 			(hide yes)
