File: hardware/pulse-wago/Link-Plug.kicad_sch (KiCad schematic)
At the start: 4 parts, among them J1901 2x05_Horizontal, U1901 THVD2442

Commit message: Rename
Parts:
- U1901: value THVD2442 -> (none); symbol V2_Interface_RS485:THVD2442 -> V2_Interface_RS485:THVD24x2; Manufacturer Texas Instruments -> (none); Mouser 595-THVD2442DRCR -> (none); Product THVD2442DRCR -> (none); Rating 20Mbps -> (none)
Other:
- note added: "Power input from plug."
- note removed: "+5V from Plug"
- note removed: "RS-422 3MHz"
- title: V2 pulse -> V2 pulse WAGO
- moved on the sheet: C1901, J1901, R1901, U1901
