File: hardware/pulse-wago/Power-Switch.kicad_sch (KiCad schematic)
At the start: 22 parts, among them J1801 WAGO 2065-100, J1802 WAGO 2065-100, U1801 BTT6010

Commit message: Rename
Connections:
- net +28V-Supply renamed +VSUPPLY
Other:
- moved on the sheet: C1806, D1801, R1809
