File: hardware/pulse-wago/pulse-wago.kicad_sch (KiCad schematic)
At the start: 44 parts, among them J101 Cortex, SW101 SKSG, SW102 SKSG, U101 TPS78433QWDRBRQ1, U102 ATSAMD51J, Y101 32k768

Commit message: Rename
Connections:
- net +5V: now also U101.6 (EN)
Other:
- sheet Link Plug: file LinkPlug.kicad_sch -> Link-Plug.kicad_sch
- sheet Link Socket: file LinkSocket.kicad_sch -> Link-Socket.kicad_sch
- sheet PWM Channel 1: file PWMChannel.kicad_sch -> PWM-Channel.kicad_sch
- sheet PWM Channel 10: file PWMChannel.kicad_sch -> PWM-Channel.kicad_sch
- sheet PWM Channel 11: file PWMChannel.kicad_sch -> PWM-Channel.kicad_sch
- sheet PWM Channel 12: file PWMChannel.kicad_sch -> PWM-Channel.kicad_sch
- sheet PWM Channel 13: file PWMChannel.kicad_sch -> PWM-Channel.kicad_sch
- sheet PWM Channel 14: file PWMChannel.kicad_sch -> PWM-Channel.kicad_sch
- sheet PWM Channel 15: file PWMChannel.kicad_sch -> PWM-Channel.kicad_sch
- sheet PWM Channel 16: file PWMChannel.kicad_sch -> PWM-Channel.kicad_sch
- sheet PWM Channel 2: file PWMChannel.kicad_sch -> PWM-Channel.kicad_sch
- sheet PWM Channel 3: file PWMChannel.kicad_sch -> PWM-Channel.kicad_sch
- sheet PWM Channel 4: file PWMChannel.kicad_sch -> PWM-Channel.kicad_sch
- sheet PWM Channel 5: file PWMChannel.kicad_sch -> PWM-Channel.kicad_sch
- sheet PWM Channel 6: file PWMChannel.kicad_sch -> PWM-Channel.kicad_sch
- sheet PWM Channel 7: file PWMChannel.kicad_sch -> PWM-Channel.kicad_sch
- sheet PWM Channel 8: file PWMChannel.kicad_sch -> PWM-Channel.kicad_sch
- sheet PWM Channel 9: file PWMChannel.kicad_sch -> PWM-Channel.kicad_sch
- sheet Power +28V: file PowerSwitch.kicad_sch -> Power-Switch.kicad_sch
Changed lines of the file:
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@@
 	(title_block
 		(title "V2 pulse WAGO")
-		(date "2026-06-08")
-		(rev "2026-06-08")
+		(date "2026-08-31")
+		(rev "2026-08-31")
 		(company "Versio Duo")
 		(comment 1 "Solenoid Controller")
@@
 			)
 		)
-		(property "Sim.Pins" "1=K 2=A"
-			(at 125.73 101.6 0)
-			(hide yes)
-			(show_name no)
-			(do_not_autoplace no)
-			(effects
-				(font
-					(size 1.27 1.27)
-				)
-			)
-		)
 		(property "Mouser" "755-SML-D12D1WT86"
 			(at 125.73 93.98 0)
@@
 			)
 		)
+		(property "Sim.Pins" "1=K 2=A"
+			(at 125.73 109.22 0)
+			(hide yes)
+			(show_name no)
+			(do_not_autoplace no)
+			(effects
+				(font
+					(size 1.27 1.27)
+				)
+			)
+		)
 		(pin "1"
 		)
@@
 		(unit 1)
 		(body_style 1)
-		(exclude_from_sim yes)
+		(exclude_from_sim no)
 		(in_bom no)
 		(on_board yes)
@@
 			)
 		)
+		(property "Sim.Enable" "0"
+			(at 184.785 170.18 0)
+			(hide yes)
+			(show_name no)
+			(do_not_autoplace no)
+			(effects
+				(font
+					(size 1.27 1.27)
+				)
+			)
+		)
 		(instances
 			(project "pulse-wago"
@@
 		(unit 1)
 		(body_style 1)
-		(exclude_from_sim yes)
+		(exclude_from_sim no)
 		(in_bom no)
 		(on_board yes)
@@
 			)
 		)
+		(property "Sim.Enable" "0"
+			(at 218.44 151.13 0)
+			(hide yes)
+			(show_name no)
+			(do_not_autoplace no)
+			(effects
+				(font
+					(size 1.27 1.27)
+				)
+			)
+		)
 		(instances
 			(project "pulse-wago"
@@
 		(unit 1)
 		(body_style 1)
-		(exclude_from_sim yes)
+		(exclude_from_sim no)
 		(in_bom no)
 		(on_board yes)
@@
 			)
 		)
+		(property "Sim.Enable" "0"
+			(at 184.785 151.765 0)
+			(hide yes)
+			(show_name no)
+			(do_not_autoplace no)
+			(effects
+				(font
+					(size 1.27 1.27)
+				)
+			)
+		)
 		(instances
 			(project "pulse-wago"
@@
 		(unit 1)
 		(body_style 1)
-		(exclude_from_sim yes)
+		(exclude_from_sim no)
 		(in_bom no)
 		(on_board yes)
@@
 			)
 		)
+		(property "Sim.Enable" "0"
+			(at 218.44 157.48 0)
+			(hide yes)
+			(show_name no)
+			(do_not_autoplace no)
+			(effects
+				(font
+					(size 1.27 1.27)
+				)
+			)
+		)
 		(instances
 			(project "pulse-wago"
@@
 		(unit 1)
 		(body_style 1)
-		(exclude_from_sim yes)
+		(exclude_from_sim no)
 		(in_bom no)
 		(on_board yes)
@@
 			)
 		)
+		(property "Sim.Enable" "0"
+			(at 158.75 161.925 0)
+			(hide yes)
+			(show_name no)
+			(do_not_autoplace no)
+			(effects
+				(font
+					(size 1.27 1.27)
+				)
+			)
+		)
 		(instances
 			(project "pulse-wago"
@@
 		(unit 1)
 		(body_style 1)
-		(exclude_from_sim yes)
+		(exclude_from_sim no)
 		(in_bom no)
 		(on_board yes)
@@
 			)
 		)
+		(property "Sim.Enable" "0"
+			(at 218.44 163.83 0)
+			(hide yes)
+			(show_name no)
+			(do_not_autoplace no)
+			(effects
+				(font
+					(size 1.27 1.27)
+				)
+			)
+		)
 		(instances
 			(project "pulse-wago"
@@
 		(unit 1)
 		(body_style 1)
-		(exclude_from_sim yes)
+		(exclude_from_sim no)
 		(in_bom no)
 		(on_board yes)
@@
 			)
 		)
+		(property "Sim.Enable" "0"
+			(at 184.785 161.29 0)
+			(hide yes)
+			(show_name no)
+			(do_not_autoplace no)
+			(effects
+				(font
+					(size 1.27 1.27)
+				)
+			)
+		)
 		(instances
 			(project "pulse-wago"
@@
 			)
 		)
-		(property "Sheetfile" "PWMChannel.kicad_sch"
+		(property "Sheetfile" "PWM-Channel.kicad_sch"
 			(at 220.98 100.9146 0)
 			(hide yes)
@@
 			)
 		)
-		(property "Sheetfile" "PWMChannel.kicad_sch"
+		(property "Sheetfile" "PWM-Channel.kicad_sch"
 			(at 193.04 84.4046 0)
 			(hide yes)
@@
 			)
 		)
-		(property "Sheetfile" "PWMChannel.kicad_sch"
+		(property "Sheetfile" "PWM-Channel.kicad_sch"
 			(at 220.98 84.4046 0)
 			(hide yes)
@@
 			)
 		)
-		(property "Sheetfile" "PWMChannel.kicad_sch"
+		(property "Sheetfile" "PWM-Channel.kicad_sch"
 			(at 248.92 100.9146 0)
 			(hide yes)
@@
 			)
 		)
-		(property "Sheetfile" "LinkSocket.kicad_sch"
+		(property "Sheetfile" "Link-Socket.kicad_sch"
 			(at 266.7 132.6646 0)
 			(hide yes)
@@
 			)
 		)
-		(property "Sheetfile" "PWMChannel.kicad_sch"
+		(property "Sheetfile" "PWM-Channel.kicad_sch"
 			(at 193.04 69.1646 0)
 			(hide yes)
@@
 			)
 		)
-		(property "Sheetfile" "PWMChannel.kicad_sch"
+		(property "Sheetfile" "PWM-Channel.kicad_sch"
 			(at 220.98 52.6546 0)
 			(hide yes)
@@
 			)
 		)
-		(property "Sheetfile" "PWMChannel.kicad_sch"
+		(property "Sheetfile" "PWM-Channel.kicad_sch"
 			(at 163.83 100.9146 0)
 			(hide yes)
@@
 			)
 		)
-		(property "Sheetfile" "PWMChannel.kicad_sch"
+		(property "Sheetfile" "PWM-Channel.kicad_sch"
 			(at 220.98 69.1646 0)
 			(hide yes)
@@
 			)
 		)
-		(property "Sheetfile" "PWMChannel.kicad_sch"
+		(property "Sheetfile" "PWM-Channel.kicad_sch"
 			(at 163.83 69.1646 0)
 			(hide yes)
@@
 			)
 		)
-		(property "Sheetfile" "PowerSwitch.kicad_sch"
+		(property "Sheetfile" "Power-Switch.kicad_sch"
 			(at 203.2 34.8746 0)
 			(hide yes)
@@
 			)
 		)
-		(property "Sheetfile" "PWMChannel.kicad_sch"
+		(property "Sheetfile" "PWM-Channel.kicad_sch"
 			(at 193.04 52.6546 0)
 			(hide yes)
@@
 			)
 		)
-		(property "Sheetfile" "PWMChannel.kicad_sch"
+		(property "Sheetfile" "PWM-Channel.kicad_sch"
 			(at 248.92 69.1646 0)
 			(hide yes)
@@
 			)
 		)
-		(property "Sheetfile" "PWMChannel.kicad_sch"
+		(property "Sheetfile" "PWM-Channel.kicad_sch"
 			(at 248.92 52.6546 0)
 			(hide yes)
@@
 			)
 		)
-		(property "Sheetfile" "LinkPlug.kicad_sch"
+		(property "Sheetfile" "Link-Plug.kicad_sch"
 			(at 227.33 127.5846 0)
 			(hide yes)
@@
 			)
 		)
-		(property "Sheetfile" "PWMChannel.kicad_sch"
+		(property "Sheetfile" "PWM-Channel.kicad_sch"
 			(at 163.83 52.6546 0)
 			(hide yes)
@@
 			)
 		)
-		(property "Sheetfile" "PWMChannel.kicad_sch"
+		(property "Sheetfile" "PWM-Channel.kicad_sch"
 			(at 193.04 100.9146 0)
 			(hide yes)
@@
 			)
 		)
-		(property "Sheetfile" "PWMChannel.kicad_sch"
+		(property "Sheetfile" "PWM-Channel.kicad_sch"
 			(at 163.83 84.4046 0)
 			(hide yes)
@@
 			)
 		)
-		(property "Sheetfile" "PWMChannel.kicad_sch"
+		(property "Sheetfile" "PWM-Channel.kicad_sch"
 			(at 248.92 84.4046 0)
 			(hide yes)
